File: PCB_evenwicht/esp32.kicad_sch (KiCad schematic)
At the start: 20 parts, among them J1 Barrel_Jack, J2 Conn_01x04_Pin, SW1 EN, SW2 FLASH, U1 ESP32-WROOM-32, U2 AMS1117-3.3, U3 MP1584

Commit message: update
Parts:
- removed C2, C4: 10uF, Capacitor_SMD:C_0805_2012Metric_Pad1.18x1.45mm_HandSolder, symbol Device:C
- removed C3: 100nF, Capacitor_SMD:C_0805_2012Metric_Pad1.18x1.45mm_HandSolder, symbol Device:C
- removed J1: Barrel_Jack, Connector_BarrelJack:BarrelJack_GCT_DCJ200-10-A_Horizontal, symbol Connector:Barrel_Jack
- removed U2: AMS1117-3.3, Package_TO_SOT_SMD:SOT-223-3_TabPin2, symbol Regulator_Linear:AMS1117-3.3
- removed U3: MP1584, Library:U1584, symbol Lib:MP1584
Connections:
- net A6: no longer names the net of U1.6 (IO34)
- net A7: no longer names the net of U1.7 (IO35)
- net VN: no longer names the net of U1.5 (SENSOR_VN)
- net VP: no longer names the net of U1.4 (SENSOR_VP)
- no-connect marks 6 -> 10
Other:
- note removed: "POWER PART"
