File: PCB_evenwicht/PCB_evenwicht.kicad_pcb (KiCad board)
At the start: 2 copper layers, 21 parts, among them IC2 A4988SETTR-T, J1 Conn_01x04_Pin, J2 Barrel_Jack, SW1 EN, SW2 FLASH, U1 ESP32-WROOM-32, U2 MP1584, U3 AMS1117-3.3

Commit message: PCB_Update
Nog enkel de footprints van de controller aanduiden en controleren van de waarden
Parts:
- removed IC2: A4988SETTR-T, A4988:QFN50P500X500X100-29N
- added IC1: A4988SETTR-T, A4988:QFN50P500X500X100-29N, F.Cu at (89.3, 41.7)
- added J3: Conn_01x04_Pin, Connector_PinHeader_2.54mm:PinHeader_1x04_P2.54mm_Vertical, F.Cu at (73.6, 51.6)
- added J4: POTy, Connector_PinHeader_2.54mm:PinHeader_1x03_P2.54mm_Vertical, F.Cu at (85.7, 52.1)
- added J5: Switchy, Connector_PinHeader_2.54mm:PinHeader_1x02_P2.54mm_Vertical, F.Cu at (78.3, 63.1)
- added JP1: MS3y, Jumper:SolderJumper-3_P1.3mm_Open_Pad1.0x1.5mm, F.Cu at (79.5, 38.1)
- added JP2: MS2y, Jumper:SolderJumper-3_P1.3mm_Open_Pad1.0x1.5mm, F.Cu at (79.5, 41.3)
- added JP3: MS1y, Jumper:SolderJumper-3_P1.3mm_Open_Pad1.0x1.5mm, F.Cu at (79.4, 45.1)
- J1: footprint Connector_PinHeader_2.00mm:PinHeader_1x04_P2.00mm_Vertical -> Connector_PinHeader_2.54mm:PinHeader_1x04_P2.54mm_Vertical
- U2: value MP1584 -> AMS1117-3.3; footprint Library:U1584 -> Package_TO_SOT_SMD:SOT-223-3_TabPin2
- U3: value AMS1117-3.3 -> MP1584; footprint Package_TO_SOT_SMD:SOT-223-3_TabPin2 -> Library:U1584
- moved U3 29.3 mm to (99.8, 52.5), turned to 0 degrees
- moved U2 28.4 mm to (105.4, 81.3), turned to 90 degrees
Connections:
- J2 pad 1: Net-(J2-Pad1) -> Vmot
- U2 pad 1: Net-(J2-Pad2) -> GND
- U2 pad 2: Net-(J2-Pad2) -> +3.3V
- U2 pad 3: Net-(J2-Pad1) -> VDD
- U3 pad 1: GND -> Net-(J2-Pad2)
- U3 pad 2: +3.3V -> Net-(J2-Pad2)
- U3 pad 3: VDD -> Vmot

Commit message: update pcb
Parts:
- added C10: 0.22uF, Capacitor_SMD:C_0603_1608Metric_Pad1.08x0.95mm_HandSolder, F.Cu at (144.3, 130.5)
- added C11: 0.1u, Capacitor_SMD:C_0603_1608Metric_Pad1.08x0.95mm_HandSolder, F.Cu at (126.0, 97.2)
- added C12: 0.22uF, Capacitor_SMD:C_0603_1608Metric_Pad1.08x0.95mm_HandSolder, F.Cu at (126.0, 99.7)
- added C13: 100nF, Capacitor_SMD:C_0603_1608Metric_Pad1.08x0.95mm_HandSolder, F.Cu at (126.0, 102.2)
- added C14: 0.1 uF, Capacitor_SMD:C_0603_1608Metric_Pad1.08x0.95mm_HandSolder, F.Cu at (126.0, 104.8)
- added C15: 4.7uF, Capacitor_SMD:C_0603_1608Metric_Pad1.08x0.95mm_HandSolder, F.Cu at (126.0, 107.3)
- added C16: 100nF, Capacitor_SMD:C_0603_1608Metric_Pad1.08x0.95mm_HandSolder, F.Cu at (126.0, 109.8)
- added C17: 4.7uF, Capacitor_SMD:C_0603_1608Metric_Pad1.08x0.95mm_HandSolder, F.Cu at (144.3, 133.0)
- added C18: 0.22uF, Capacitor_SMD:C_0603_1608Metric_Pad1.08x0.95mm_HandSolder, F.Cu at (126.0, 112.3)
- added C5: 0.1u, Capacitor_SMD:C_0603_1608Metric_Pad1.08x0.95mm_HandSolder, F.Cu at (144.3, 117.9)
- added C6: 0.22uF, Capacitor_SMD:C_0603_1608Metric_Pad1.08x0.95mm_HandSolder, F.Cu at (144.3, 120.4)
- added C7: 100nF, Capacitor_SMD:C_0603_1608Metric_Pad1.08x0.95mm_HandSolder, F.Cu at (144.3, 123.0)
- added C8: 0.1 uF, Capacitor_SMD:C_0603_1608Metric_Pad1.08x0.95mm_HandSolder, F.Cu at (144.3, 125.5)
- added C9: 100nF, Capacitor_SMD:C_0603_1608Metric_Pad1.08x0.95mm_HandSolder, F.Cu at (144.3, 128.0)
- added IC2: A4988SETTR-T, A4988:QFN50P500X500X100-29N, F.Cu at (136.5, 111.5)
- added J6: Conn_01x04_Pin, Connector_PinHeader_2.54mm:PinHeader_1x04_P2.54mm_Vertical, F.Cu at (130.5, 98.3)
- added J7: Switchx, Connector_PinHeader_2.54mm:PinHeader_1x02_P2.54mm_Vertical, F.Cu at (144.5, 98.3)
- added J8: POTx, Connector_PinHeader_2.54mm:PinHeader_1x03_P2.54mm_Vertical, F.Cu at (150.1, 105.5)
- added J9: Switch_einde, Connector_PinHeader_2.54mm:PinHeader_1x02_P2.54mm_Vertical, F.Cu at (149.1, 98.3)
- added JP4: MS3x, Jumper:SolderJumper-3_P1.3mm_Open_Pad1.0x1.5mm, F.Cu at (145.0, 105.0)
- added JP5: MS2x, Jumper:SolderJumper-3_P1.3mm_Open_Pad1.0x1.5mm, F.Cu at (145.0, 108.8)
- added JP6: MS1x, Jumper:SolderJumper-3_P1.3mm_Open_Pad1.0x1.5mm, F.Cu at (145.0, 112.6)
- added R10: 50m, Resistor_SMD:R_0805_2012Metric_Pad1.20x1.40mm_HandSolder, F.Cu at (148.9, 124.0)
- added R11: 50m, Resistor_SMD:R_0805_2012Metric_Pad1.20x1.40mm_HandSolder, F.Cu at (148.9, 127.0)
- added R12: 100K, Resistor_SMD:R_0805_2012Metric_Pad1.20x1.40mm_HandSolder, F.Cu at (135.2, 97.5)
- added R13: 25K, Resistor_SMD:R_0805_2012Metric_Pad1.20x1.40mm_HandSolder, F.Cu at (135.2, 100.4)
- added R14: 50m, Resistor_SMD:R_0805_2012Metric_Pad1.20x1.40mm_HandSolder, F.Cu at (135.2, 103.3)
- added R15: 50m, Resistor_SMD:R_0805_2012Metric_Pad1.20x1.40mm_HandSolder, F.Cu at (135.2, 106.3)
- added R8: 100K, Resistor_SMD:R_0805_2012Metric_Pad1.20x1.40mm_HandSolder, F.Cu at (148.9, 118.2)
- added R9: 25K, Resistor_SMD:R_0805_2012Metric_Pad1.20x1.40mm_HandSolder, F.Cu at (148.9, 121.1)
- J1: value Conn_01x04_Pin -> Barrel_Jack; footprint Connector_PinHeader_2.54mm:PinHeader_1x04_P2.54mm_Vertical -> Connector_BarrelJack:BarrelJack_GCT_DCJ200-10-A_Horizontal
- J2: value Barrel_Jack -> Conn_01x04_Pin; footprint Connector_BarrelJack:BarrelJack_GCT_DCJ200-10-A_Horizontal -> Connector_PinHeader_2.54mm:PinHeader_1x04_P2.54mm_Vertical
- J3: value Conn_01x04_Pin -> Switchy; footprint Connector_PinHeader_2.54mm:PinHeader_1x04_P2.54mm_Vertical -> Connector_PinHeader_2.54mm:PinHeader_1x02_P2.54mm_Vertical
- J4: value POTy -> Conn_01x04_Pin; footprint Connector_PinHeader_2.54mm:PinHeader_1x03_P2.54mm_Vertical -> Connector_PinHeader_2.54mm:PinHeader_1x04_P2.54mm_Vertical
- J5: value Switchy -> POTy; footprint Connector_PinHeader_2.54mm:PinHeader_1x02_P2.54mm_Vertical -> Connector_PinHeader_2.54mm:PinHeader_1x03_P2.54mm_Vertical
Connections:
- net /EN renamed /ESP32/EN
- net MS1 renamed MS1_1
- net MS2 renamed MS2_1
- net MS3 renamed MS3_1
- J1 pad 1: +3.3V -> Vmot
- J1 pad 2: RX0 -> Net-(J1-Pad2)
- J1 pad 3: TX0 -> (no net)
- J2 pad 1: Vmot -> +3.3V
- J2 pad 2: Net-(J2-Pad2) -> RX0
- J2 pad 3: (no net) -> TX0
- J3 pad 1: Net-(IC1-OUT2B) -> GPIO4
- J3 pad 2: Net-(IC1-OUT2A) -> GND
- J4 pad 1: GND -> Net-(IC1-OUT2B)
- J4 pad 2: REF1 -> Net-(IC1-OUT2A)
- J4 pad 3: +3.3V -> Net-(IC1-OUT1A)
- J5 pad 1: GPIO4 -> GND
- J5 pad 2: GND -> REF1
- U1 pad 4: VP -> unconnected-(U1-SENSOR_VP-Pad4)
- U1 pad 5: VN -> unconnected-(U1-SENSOR_VN-Pad5)
- U1 pad 6: A6 -> unconnected-(U1-IO34-Pad6)
- U1 pad 7: A7 -> unconnected-(U1-IO35-Pad7)
- U3 pad 1: Net-(J2-Pad2) -> Net-(J1-Pad2)
- U3 pad 2: Net-(J2-Pad2) -> Net-(J1-Pad2)

Commit message: klj
Parts:
- moved J3 73.2 mm to (141.6, 78.7)
- moved J6 59.9 mm to (181.0, 66.0), turned to 90 degrees
- moved IC2 53.0 mm to (181.4, 83.4)
- moved J5 39.3 mm to (95.9, 27.9)
- moved J2 27.7 mm to (120.7, 90.8), turned to 90 degrees
- moved J9 20.0 mm to (153.0, 78.7)
- moved J7 19.8 mm to (147.3, 78.7)
- moved J8 11.8 mm to (161.9, 105.5)
Connections:
- IC2 pad 10: MS2_1 -> MS2_2
- IC2 pad 11: MS3_1 -> MS3_2
- IC2 pad 16: GPIO19 -> A4
- IC2 pad 17: REF1 -> REF2
- IC2 pad 19: GPIO18 -> A5
- IC2 pad 9: MS1_1 -> MS1_2
- JP4 pad 2: MS3_1 -> MS3_2
- JP5 pad 2: MS2_1 -> MS2_2
- JP6 pad 2: MS1_1 -> MS1_2
Changed lines of the file:
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@@
   (net 77 "unconnected-(U1-IO34-Pad6)")
   (net 78 "unconnected-(U1-IO35-Pad7)")
+  (net 79 "MS1_2")
+  (net 80 "MS2_2")
+  (net 81 "MS3_2")
   (footprint "Resistor_SMD:R_0805_2012Metric_Pad1.20x1.40mm_HandSolder" (layer "F.Cu")
     (at 135.16 103.35)
@@
   )
   (footprint "Connector_PinHeader_2.54mm:PinHeader_1x03_P2.54mm_Vertical" (layer "F.Cu")
-    (at 150.11 105.5)
+    (at 161.925 105.5)
     (descr "Through hole straight pin header, 1x03, 2.54mm pitch, single row")
     (tags "Through hole pin header THT 1x03 2.54mm single row")
@@
       (net 2 "GND") (pinfunction "A") (pintype "passive"))
     (pad "2" smd rect (at 0 0) (size 1 1.5) (layers "F.Cu" "F.Mask")
-      (net 15 "MS1_1") (pinfunction "C") (pintype "passive"))
+      (net 79 "MS1_2") (pinfunction "C") (pintype "passive"))
     (pad "3" smd rect (at 1.3 0) (size 1 1.5) (layers "F.Cu" "F.Mask")
       (net 1 "+3.3V") (pinfunction "B") (pintype "passive"))
@@
       (net 2 "GND") (pinfunction "A") (pintype "passive"))
     (pad "2" smd rect (at 0 0) (size 1 1.5) (layers "F.Cu" "F.Mask")
-      (net 46 "MS2_1") (pinfunction "C") (pintype "passive"))
+      (net 80 "MS2_2") (pinfunction "C") (pintype "passive"))
     (pad "3" smd rect (at 1.3 0) (size 1 1.5) (layers "F.Cu" "F.Mask")
       (net 1 "+3.3V") (pinfunction "B") (pintype "passive"))
   )
   (footprint "Connector_PinHeader_2.54mm:PinHeader_1x04_P2.54mm_Vertical" (layer "F.Cu")
-    (at 94.615 81.28 -90)
+    (at 120.66 90.805 90)
     (descr "Through hole straight pin header, 1x04, 2.54mm pitch, single row")
     (tags "Through hole pin header THT 1x04 2.54mm single row")
@@
     (property "ki_keywords" "connector")
     (attr through_hole)
-    (fp_text reference "J2" (at 0 -2.33 -90) (layer "F.SilkS")
-        (effects (font (size 1 1) (thickness 0.15)))
-    )
-    (fp_text value "Conn_01x04_Pin" (at 0 9.95 -90) (layer "F.Fab")
+    (fp_text reference "J2" (at 0 -2.33 90) (layer "F.SilkS")
+        (effects (font (size 1 1) (thickness 0.15)))
+    )
+    (fp_text value "Conn_01x04_Pin" (at 0 9.95 90) (layer "F.Fab")
         (effects (font (size 1 1) (thickness 0.15)))
     )
@@
     (fp_line (start 1.27 8.89) (end -1.27 8.89)
       (stroke (width 0.1) (type solid)) (layer "F.Fab"))
-    (pad "1" thru_hole rect (at 0 0 270) (size 1.7 1.7) (drill 1) (layers "*.Cu" "*.Mask")
+    (pad "1" thru_hole rect (at 0 0 90) (size 1.7 1.7) (drill 1) (layers "*.Cu" "*.Mask")
       (net 1 "+3.3V") (pinfunction "Pin_1") (pintype "passive"))
-    (pad "2" thru_hole oval (at 0 2.54 270) (size 1.7 1.7) (drill 1) (layers "*.Cu" "*.Mask")
+    (pad "2" thru_hole oval (at 0 2.54 90) (size 1.7 1.7) (drill 1) (layers "*.Cu" "*.Mask")
       (net 7 "RX0") (pinfunction "Pin_2") (pintype "passive"))
-    (pad "3" thru_hole oval (at 0 5.08 270) (size 1.7 1.7) (drill 1) (layers "*.Cu" "*.Mask")
+    (pad "3" thru_hole oval (at 0 5.08 90) (size 1.7 1.7) (drill 1) (layers "*.Cu" "*.Mask")
       (net 8 "TX0") (pinfunction "Pin_3") (pintype "passive"))
-    (pad "4" thru_hole oval (at 0 7.62 270) (size 1.7 1.7) (drill 1) (layers "*.Cu" "*.Mask")
+    (pad "4" thru_hole oval (at 0 7.62 90) (size 1.7 1.7) (drill 1) (layers "*.Cu" "*.Mask")
       (net 2 "GND") (pinfunction "Pin_4") (pintype "passive"))
     (model "${KICAD6_3DMODEL_DIR}/Connector_PinHeader_2.54mm.3dshapes/PinHeader_1x04_P2.54mm_Vertical.wrl"
@@
       (net 2 "GND") (pinfunction "A") (pintype "passive"))
     (pad "2" smd rect (at 0 0) (size 1 1.5) (layers "F.Cu" "F.Mask")
-      (net 47 "MS3_1") (pinfunction "C") (pintype "passive"))
+      (net 81 "MS3_2") (pinfunction "C") (pintype "passive"))
     (pad "3" smd rect (at 1.3 0) (size 1 1.5) (layers "F.Cu" "F.Mask")
       (net 1 "+3.3V") (pinfunction "B") (pintype "passive"))
@@
   )
   (footprint "Connector_PinHeader_2.54mm:PinHeader_1x02_P2.54mm_Vertical" (layer "F.Cu")
-    (at 144.46 98.3)
+    (at 147.32 78.74)
     (descr "Through hole straight pin header, 1x02, 2.54mm pitch, single row")
     (tags "Through hole pin header THT 1x02 2.54mm single row")
@@
   )
   (footprint "Connector_PinHeader_2.54mm:PinHeader_1x04_P2.54mm_Vertical" (layer "F.Cu")
-    (at 130.46 98.3)
+    (at 180.975 66.04 90)
     (descr "Through hole straight pin header, 1x04, 2.54mm pitch, single row")
     (tags "Through hole pin header THT 1x04 2.54mm single row")
@@
     (property "ki_keywords" "connector")
     (attr through_hole)
-    (fp_text reference "J6" (at 0 -2.33) (layer "F.SilkS")
-        (effects (font (size 1 1) (thickness 0.15)))
-    )
-    (fp_text value "Conn_01x04_Pin" (at 0 9.95) (layer "F.Fab")
-        (effects (font (size 1 1) (thickness 0.15)))
-    )
-    (fp_text user "${REFERENCE}" (at 0 3.81 90) (layer "F.Fab")
+    (fp_text reference "J6" (at 0 -2.33 90) (layer "F.SilkS")
+        (effects (font (size 1 1) (thickness 0.15)))
+    )
+    (fp_text value "Conn_01x04_Pin" (at 0 9.95 90) (layer "F.Fab")
+        (effects (font (size 1 1) (thickness 0.15)))
+    )
+    (fp_text user "${REFERENCE}" (at 0 3.81) (layer "F.Fab")
         (effects (font (size 1 1) (thickness 0.15)))
     )
@@
     (fp_line (start 1.27 8.89) (end -1.27 8.89)
       (stroke (width 0.1) (type solid)) (layer "F.Fab"))
-    (pad "1" thru_hole rect (at 0 0) (size 1.7 1.7) (drill 1) (layers "*.Cu" "*.Mask")
+    (pad "1" thru_hole rect (at 0 0 90) (size 1.7 1.7) (drill 1) (layers "*.Cu" "*.Mask")
       (net 48 "Net-(IC2-OUT2B)") (pinfunction "Pin_1") (pintype "passive"))
-    (pad "2" thru_hole oval (at 0 2.54) (size 1.7 1.7) (drill 1) (layers "*.Cu" "*.Mask")
+    (pad "2" thru_hole oval (at 0 2.54 90) (size 1.7 1.7) (drill 1) (layers "*.Cu" "*.Mask")
       (net 69 "Net-(IC2-OUT2A)") (pinfunction "Pin_2") (pintype "passive"))
-    (pad "3" thru_hole oval (at 0 5.08) (size 1.7 1.7) (drill 1) (layers "*.Cu" "*.Mask")
+    (pad "3" thru_hole oval (at 0 5.08 90) (size 1.7 1.7) (drill 1) (layers "*.Cu" "*.Mask")
       (net 67 "Net-(IC2-OUT1A)") (pinfunction "Pin_3") (pintype "passive"))
-    (pad "4" thru_hole oval (at 0 7.62) (size 1.7 1.7) (drill 1) (layers "*.Cu" "*.Mask")
+    (pad "4" thru_hole oval (at 0 7.62 90) (size 1.7 1.7) (drill 1) (layers "*.Cu" "*.Mask")
       (net 65 "Net-(IC2-OUT1B)") (pinfunction "Pin_4") (pintype "passive"))
     (model "${KICAD6_3DMODEL_DIR}/Connector_PinHeader_2.54mm.3dshapes/PinHeader_1x04_P2.54mm_Vertical.wrl"
@@
   )
   (footprint "Connector_PinHeader_2.54mm:PinHeader_1x02_P2.54mm_Vertical" (layer "F.Cu")
-    (at 73.63 51.585)
+    (at 141.605 78.735)
     (descr "Through hole straight pin header, 1x02, 2.54mm pitch, single row")
     (tags "Through hole pin header THT 1x02 2.54mm single row")
@@
   )
   (footprint "Connector_PinHeader_2.54mm:PinHeader_1x02_P2.54mm_Vertical" (layer "F.Cu")
-    (at 149.11 98.3)
+    (at 153.035 78.735)
     (descr "Through hole straight pin header, 1x02, 2.54mm pitch, single row")
     (tags "Through hole pin header THT 1x02 2.54mm single row")
@@
   )
   (footprint "A4988:QFN50P500X500X100-29N" (layer "F.Cu")
-    (at 136.46 111.45)
+    (at 181.38 83.375)
     (descr "<b>ET Package, 28-Pin QFN with Exposed Thermal Pad</b><br>")
     (property "DESCRIPTION" "DMOS Microstepping Driver with Translator  and Overcurrent Protection")
@@
       (net 13 "Net-(IC2-VREG)") (pinfunction "VREG") (pintype "bidirectional"))
     (pad "9" smd rect (at -1 2.35 90) (size 1.15 0.3) (layers "F.Cu" "F.Paste" "F.Mask")
-      (net 15 "MS1_1") (pinfunction "MS1") (pintype "bidirectional"))
+      (net 79 "MS1_2") (pinfunction "MS1") (pintype "bidirectional"))
     (pad "10" smd rect (at -0.5 2.35 90) (size 1.15 0.3) (layers "F.Cu" "F.Paste" "F.Mask")
-      (net 46 "MS2_1") (pinfunction "MS2") (pintype "bidirectional"))
+      (net 80 "MS2_2") (pinfunction "MS2") (pintype "bidirectional"))
     (pad "11" smd rect (at 0 2.35 90) (size 1.15 0.3) (layers "F.Cu" "F.Paste" "F.Mask")
-      (net 47 "MS3_1") (pinfunction "MS3") (pintype "bidirectional"))
+      (net 81 "MS3_2") (pinfunction "MS3") (pintype "bidirectional"))
     (pad "12" smd rect (at 0.5 2.35 90) (size 1.15 0.3) (layers "F.Cu" "F.Paste" "F.Mask")
       (net 49 "!RESET") (pinfunction "~{RESET}") (pintype "bidirectional"))
@@
       (net 3 "VDD") (pinfunction "VDD") (pintype "bidirectional"))
     (pad "16" smd rect (at 2.35 1) (size 1.15 0.3) (layers "F.Cu" "F.Paste" "F.Mask")
-      (net 35 "GPIO19") (pinfunction "STEP") (pintype "bidirectional"))
+      (net 16 "A4") (pinfunction "STEP") (pintype "bidirectional"))
     (pad "17" smd rect (at 2.35 0.5) (size 1.15 0.3) (layers "F.Cu" "F.Paste" "F.Mask")
-      (net 52 "REF1") (pinfunction "REF") (pintype "bidirectional"))
+      (net 73 "REF2") (pinfunction "REF") (pintype "bidirectional"))
     (pad "18" smd rect (at 2.35 0) (size 1.15 0.3) (layers "F.Cu" "F.Paste" "F.Mask")
       (net 2 "GND") (pinfunction "GND_2") (pintype "bidirectional"))
     (pad "19" smd rect (at 2.35 -0.5) (size 1.15 0.3) (layers "F.Cu" "F.Paste" "F.Mask")
-      (net 34 "GPIO18") (pinfunction "DIR") (pintype "bidirectional"))
+      (net 17 "A5") (pinfunction "DIR") (pintype "bidirectional"))
     (pad "20" smd rect (at 2.35 -1) (size 1.15 0.3) (layers "F.Cu" "F.Paste" "F.Mask")
       (net 64 "unconnected-(IC2-NC_2-Pad20)") (pinfunction "NC_2") (pintype "bidirectional+no_connect"))
@@
   )
   (footprint "Connector_PinHeader_2.54mm:PinHeader_1x03_P2.54mm_Vertical" (layer "F.Cu")
-    (at 78.28 63.085)
+    (at 95.885 27.94)
     (descr "Through hole straight pin header, 1x03, 2.54mm pitch, single row")
     (tags "Through hole pin header THT 1x03 2.54mm single row")

Commit message: Update_Update
PCB eens snel geroute
Parts:
- C10, C11, C12, C13, C14, C16, C18, C5, C6, C7, C8, C9: footprint Capacitor_SMD:C_0603_1608Metric_Pad1.08x0.95mm_HandSolder -> Capacitor_SMD:C_0805_2012Metric_Pad1.18x1.45mm_HandSolder
- C15, C17: footprint Capacitor_SMD:C_0603_1608Metric_Pad1.08x0.95mm_HandSolder -> Capacitor_SMD:C_1206_3216Metric_Pad1.33x1.80mm_HandSolder
- moved JP1 91.3 mm to (109.2, 124.4), turned to 90 degrees
- moved JP2 87.1 mm to (105.4, 124.4), turned to 90 degrees
- moved J5 85.2 mm to (119.4, 109.9)
- moved JP3 82.3 mm to (101.0, 124.5), turned to 90 degrees
- moved IC1 74.2 mm to (104.8, 114.3)
- moved J1 71.5 mm to (75.0, 77.1), turned to 0 degrees
- moved J4 50.0 mm to (101.0, 99.7), turned to 90 degrees
- moved R10 49.6 mm to (102.9, 105.4), turned to 90 degrees
- moved C5 48.6 mm to (95.9, 114.3), turned to 90 degrees
- moved C6 47.3 mm to (97.2, 124.2), turned to -90 degrees
- moved C8 47.1 mm to (97.8, 118.3), turned to -90 degrees
- moved C9 46.9 mm to (101.6, 108.6), turned to 180 degrees
- moved R11 46.8 mm to (107.3, 105.4), turned to 90 degrees
- moved J6 44.8 mm to (150.7, 99.1)
- moved J9 43.7 mm to (110.7, 67.6), turned to -90 degrees
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Connections:
- C10 pad 1: VDD -> +3.3V
- C18 pad 1: VDD -> +3.3V
- IC1 pad 15: VDD -> +3.3V
- IC2 pad 15: VDD -> +3.3V
Routing:
- net +3.3V: track 0.00 -> 344.6 mm, vias 0 -> 12
- net Vmot: track 0.00 -> 185.3 mm, vias 0 -> 8
- net GND: track 0.00 -> 30.0 mm, vias 0 -> 20
- net !SLEEP: track 0.00 -> 25.4 mm
- net VDD: track 0.00 -> 23.9 mm
- net GPIO18: track 0.00 -> 18.6 mm
- net Net-(IC1-OUT1B): track 0.00 -> 16.1 mm
- net Net-(IC2-OUT2B): track 0.00 -> 14.8 mm
- net Net-(IC1-OUT2B): track 0.00 -> 14.8 mm
- net Net-(IC2-OUT1B): track 0.00 -> 14.3 mm
- net TX0: track 0.00 -> 13.8 mm
- net Net-(J1-Pad2): track 0.00 -> 13.6 mm
- net REF1: track 0.00 -> 13.3 mm
- net RX0: track 0.00 -> 13.1 mm
- net Net-(IC1-OUT2A): track 0.00 -> 12.6 mm
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- added copper zone on B.Cu, net GND
- added copper zone on F.Cu, net GND

Commit message: fdq
Parts:
- added RV1: R_Potentiometer, Potentiometer_THT:Potentiometer_Bourns_3386P_Vertical, F.Cu at (164.8, 87.9)
- added RV2: R_Potentiometer, Potentiometer_THT:Potentiometer_Bourns_3386P_Vertical, F.Cu at (151.1, 87.9)
- moved C5 89.3 mm to (162.9, 55.2), turned to 0 degrees
- moved C6 87.8 mm to (153.0, 56.5), turned to 180 degrees
- moved C8 86.5 mm to (158.9, 57.1), turned to 180 degrees
- moved J4 86.1 mm to (177.5, 60.3), turned to 0 degrees
- moved JP3 82.4 mm to (152.7, 60.3), turned to 0 degrees
- moved C9 82.2 mm to (168.6, 61.0), turned to 90 degrees
- moved R10 81.3 mm to (171.8, 62.2), turned to 0 degrees
- moved J8 79.8 mm to (88.6, 97.5), turned to 180 degrees
- moved IC1 76.8 mm to (162.9, 64.1), turned to -90 degrees
- moved JP2 76.2 mm to (152.8, 64.8), turned to 0 degrees
- moved R11 75.2 mm to (171.8, 66.7), turned to 0 degrees
- moved C7 73.4 mm to (168.6, 67.3), turned to 90 degrees
- moved JP1 70.8 mm to (152.8, 68.6), turned to 0 degrees
- moved C10 67.4 mm to (159.5, 71.1), turned to 180 degrees
- moved R9 65.5 mm to (152.5, 72.4), turned to 0 degrees
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Connections:
- IC1 pad 12: !RESET -> GND
- IC1 pad 14: !SLEEP -> GND
- IC1 pad 17: REF1 -> Net-(IC1-REF)
- IC2 pad 12: !RESET -> GND
- IC2 pad 14: !SLEEP -> GND
- IC2 pad 17: REF2 -> Net-(IC2-REF)
- J3 pad 1: GPIO4 -> GPIO14
- J5 pad 2: REF1 -> A9
- J7 pad 1: GPIO14 -> GPIO27
- J8 pad 2: REF2 -> A8
- J9 pad 1: GPIO27 -> GPIO12
- R12 pad 1: !SLEEP -> GND
- R8 pad 1: !SLEEP -> GND
Routing:
- net +3.3V: track 344.6 -> 260.4 mm, vias 12 -> 13
- net GND: track 30.0 -> 81.2 mm, vias 20 -> 12
- net A8: track 0.00 -> 45.6 mm, vias 0 -> 1
- net A5: track 0.00 -> 44.2 mm, vias 0 -> 2
- net A4: track 0.00 -> 39.6 mm, vias 0 -> 2
- net A9: track 0.00 -> 39.2 mm, vias 0 -> 1
- net GPIO19: track 4.11 -> 43.0 mm, vias 0 -> 2
- net Net-(IC2-REF): track 0.00 -> 33.6 mm
- net GPIO27: track 5.74 -> 35.7 mm, vias 0 -> 1
- net GPIO18: track 18.6 -> 48.5 mm, vias 0 -> 2
- net GPIO12: track 0.00 -> 28.8 mm, vias 0 -> 1
- net Net-(IC1-REF): track 0.00 -> 26.0 mm
- net GPIO14: track 6.62 -> 32.3 mm, vias 0 -> 1
- net !SLEEP: track 25.4 -> 0.00 mm
- net REF1: track 13.3 -> 0.00 mm
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Other:
- board outline added: 95 x 59.9 mm
- board text added: "Plop En kwebbel"

Commit message: fdqjmlk
Parts:
- removed R12, R8: 100K, Resistor_SMD:R_0805_2012Metric_Pad1.20x1.40mm_HandSolder
- added C19: 47uF, Capacitor_SMD:CP_Elec_6.3x5.9, F.Cu at (150.1, 94.0)
- added C20: 47uF, Capacitor_SMD:CP_Elec_6.3x5.9, F.Cu at (150.1, 58.4)
- moved U3 58.0 mm to (124.6, 101.9), turned to 180 degrees
- moved JP6 48.9 mm to (164.8, 72.5), turned to -90 degrees
- moved C12 46.9 mm to (164.5, 76.6), turned to 0 degrees
- moved JP5 46.5 mm to (161.0, 72.5), turned to -90 degrees
- moved JP4 44.9 mm to (157.4, 72.5), turned to -90 degrees
- moved R13 43.3 mm to (154.1, 72.8), turned to -90 degrees
- moved C14 42.3 mm to (167.3, 80.1)
- moved J1 39.5 mm to (139.2, 87.9), turned to 0 degrees
- moved C11 38.1 mm to (167.4, 83.2), turned to 180 degrees
- moved C18 34.3 mm to (154.4, 78.0), turned to 90 degrees
- moved IC2 32.0 mm to (160.5, 81.9), turned to 180 degrees
- moved C13 28.3 mm to (163.5, 87.6), turned to 180 degrees
- moved J8 25.7 mm to (107.7, 80.3), turned to 90 degrees
- moved R14 24.7 mm to (163.5, 90.8)
- moved RV1 24.4 mm to (145.8, 72.6), turned to 0 degrees
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Connections:
- IC1 pad 14: GND -> +3.3V
- IC1 pad 29: unconnected-(IC1-EP-Pad29) -> GND
- IC2 pad 14: GND -> +3.3V
- IC2 pad 29: unconnected-(IC2-EP-Pad29) -> GND
Routing:
- net +3.3V: track 260.4 -> 194.9 mm, vias 13 -> 12
- net Vmot: track 183.2 -> 135.9 mm
- net VDD: track 16.8 -> 55.2 mm
- net A8: track 45.6 -> 18.4 mm
- net Net-(IC2-REF): track 33.6 -> 12.4 mm
- net GPIO18: track 48.5 -> 31.4 mm
- net A9: track 39.2 -> 23.1 mm
- net Net-(J1-Pad2): track 12.6 -> 24.8 mm
- net GPIO19: track 43.0 -> 32.4 mm
- net GPIO27: track 35.7 -> 25.5 mm
- net Net-(IC2-OUT1B): track 15.0 -> 24.9 mm
- net A4: track 39.6 -> 49.4 mm
- net Net-(IC1-OUT2B): track 15.4 -> 5.93 mm
- net Net-(IC1-OUT1B): track 15.2 -> 23.2 mm
- net Net-(IC2-OUT2B): track 13.8 -> 6.29 mm
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Other:
- board size 95 x 59.9 mm -> 66.5 x 56.6 mm
- board text added: "12V"
- board text added: "Emiel Dever & Jonathan Gheysens IB3 V1"
- board text added: "S_bal"
- board text added: "VIN"
- board text added: "X"
- board text added: "Y"
- board text removed: "Plop En kwebbel"
