File: PCB_evenwicht/PCB_evenwicht.kicad_pcb (KiCad board)
At the start: 2 copper layers, 66.5 x 56.6 mm, 59 parts, among them IC1 A4988SETTR-T, IC2 A4988SETTR-T, J1 Barrel_Jack, J2 Conn_01x04_Pin, J3 Switchy, J4 Conn_01x04_Pin, J5 POTy, J6 Conn_01x04_Pin, J7 Switchx, J8 POTx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

Commit message: dqfsjmkmlqfd
Parts:
- JP1: value MS3y -> MS3
- JP2: value MS2y -> MS2
- JP3: value MS1y -> MS1
- JP4: value MS3x -> MS3
- JP5: value MS2x -> MS2
- JP6: value MS1x -> MS1
- moved R5 1.04 mm to (137.9, 56.7), turned to -90 degrees
- moved J6 0.55 mm to (168.4, 86.6)
- moved U3 0.28 mm to (124.9, 101.9)
Routing:
- net Net-(J1-Pad2): track 24.8 -> 18.4 mm
- net TX0: track 10.5 -> 9.55 mm
- net Net-(IC2-OUT2B): track 6.29 -> 6.84 mm
- net Net-(IC2-OUT1B): track 24.9 -> 25.5 mm
- net Net-(IC2-OUT1A): track 17.5 -> 18.0 mm
- net GND: vias 30 -> 34
Other:
- outline, holes or cut-outs redrawn

Commit message: goed
Parts:
- C15, C17: footprint Capacitor_SMD:C_1206_3216Metric_Pad1.33x1.80mm_HandSolder -> Capacitor_SMD:C_0805_2012Metric_Pad1.18x1.45mm_HandSolder
- moved RV2 1.01 mm to (144.8, 83.3)
- moved SW2 0.66 mm to (136.3, 78.2)
- moved RV1 0.16 mm to (145.9, 72.7)
Connections:
- IC1 pad 12: GND -> +3.3V
- IC2 pad 12: GND -> +3.3V
Routing:
- net +3.3V: track 195.2 -> 205.2 mm, vias 12 -> 16
- net GND: track 85.7 -> 80.2 mm
- net Net-(IC2-REF): track 12.1 -> 10.9 mm
Other:
- board text added: "Emiel Dever & Jonathan Gheysens IB3 V1.1"
- board text removed: "Emiel Dever & Jonathan Gheysens IB3 V1"
