File: PCB_evenwicht/a4988_1.kicad_sch (KiCad schematic)
At the start: 12 parts, among them IC1 A4988SETTR-T, J4 Conn_01x04_Pin

Commit message: update
Connections:
- no-connect marks 3 -> 4
Changed lines of the file:
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@@
   (junction (at 135.89 59.69) (diameter 0) (color 0 0 0 0)
   )
+  (no_connect (at 64.77 97.79))
   (no_connect (at 80.01 107.95))
   (no_connect (at 85.09 107.95))

Commit message: update pcb-design
Parts:
- added C17: 4.7uF, symbol Device:C
- C7, C9: value 100uF -> 100nF
Connections:
- net GND: now also C17.1
- net Vmot: now also C17.2
Other:
- note removed: "NOG een 4.7uf condensator denk ik ergens plaatsen"
Changed lines of the file:
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@@
   (junction (at 107.95 49.53) (diameter 0) (color 0 0 0 0)
   )
+  (junction (at 107.95 45.72) (diameter 0) (color 0 0 0 0)
+  )
   (junction (at 116.84 105.41) (diameter 0) (color 0 0 0 0)
   )
@@
   )
   (junction (at 135.89 59.69) (diameter 0) (color 0 0 0 0)
+  )
+  (junction (at 121.92 45.72) (diameter 0) (color 0 0 0 0)
   )
   (no_connect (at 64.77 97.79))
@@
     (stroke (width 0) (type default))
   )
+  (wire (pts (xy 121.92 45.72) (xy 137.16 45.72))
+    (stroke (width 0) (type default))
+  )
   (wire (pts (xy 107.95 49.53) (xy 107.95 52.07))
     (stroke (width 0) (type default))
@@
     (stroke (width 0) (type default))
   )
-  (wire (pts (xy 107.95 49.53) (xy 115.57 49.53))
+  (wire (pts (xy 107.95 45.72) (xy 121.92 45.72))
     (stroke (width 0) (type default))
   )
@@
   (wire (pts (xy 121.92 90.17) (xy 102.87 90.17))
     (stroke (width 0) (type default))
-  )
-  (text "NOG een 4.7uf condensator denk ik ergens plaatsen\n"
-    (at 113.03 87.63 0)
-    (effects (font (size 1.27 1.27)) (justify left bottom))
   )
   (global_label "GPIO18" (shape input) (at 64.77 59.69 180) (fields_autoplaced)
@@
     )
   )
-  (global_label "Vmot" (shape input) (at 115.57 49.53 0) (fields_autoplaced)
+  (global_label "Vmot" (shape input) (at 137.16 45.72 0) (fields_autoplaced)
     (effects (font (size 1.27 1.27)) (justify left))
-    (property "Intersheetrefs" "${INTERSHEET_REFS}" (at 123.1324 49.53 0)
+    (property "Intersheetrefs" "${INTERSHEET_REFS}" (at 144.7224 45.72 0)
       (effects (font (size 1.27 1.27)) (justify left) hide)
     )
@@
       (effects (font (size 1.27 1.27)))
     )
-    (property "Value" "100uF" (at 128.27 49.53 90)
+    (property "Value" "100nF" (at 128.27 49.53 90)
       (effects (font (size 1.27 1.27)))
     )
@@
         (path "/1568d5f0-bcdb-494d-bbf5-b93d65138b4f/de18e6c3-6c35-4eb3-86ab-f4d9b06c1c30"
           (reference "J4") (unit 1)
+        )
+      )
+    )
+  )
+  (symbol (lib_id "Device:C") (at 121.92 41.91 0) (unit 1)
+    (in_bom yes) (on_board yes) (dnp no) (fields_autoplaced)
+    (property "Reference" "C17" (at 125.73 41.275 0)
+      (effects (font (size 1.27 1.27)) (justify left))
+    )
+    (property "Value" "4.7uF" (at 125.73 43.815 0)
+      (effects (font (size 1.27 1.27)) (justify left))
+    )
+    (property "Footprint" "" (at 122.8852 45.72 0)
+      (effects (font (size 1.27 1.27)) hide)
+    )
+    (property "Datasheet" "~" (at 121.92 41.91 0)
+      (effects (font (size 1.27 1.27)) hide)
+    )
+    (pin "1")
+    (pin "2")
+    (instances
+      (project "PCB_evenwicht"
+        (path "/1568d5f0-bcdb-494d-bbf5-b93d65138b4f/de18e6c3-6c35-4eb3-86ab-f4d9b06c1c30"
+          (reference "C17") (unit 1)
         )
       )
@@
     )
   )
+  (symbol (lib_id "power:GND") (at 121.92 38.1 180) (unit 1)
+    (in_bom yes) (on_board yes) (dnp no) (fields_autoplaced)
+    (property "Reference" "#PWR033" (at 121.92 31.75 0)
+      (effects (font (size 1.27 1.27)) hide)
+    )
+    (property "Value" "GND" (at 121.92 34.29 0)
+      (effects (font (size 1.27 1.27)))
+    )
+    (property "Footprint" "" (at 121.92 38.1 0)
+      (effects (font (size 1.27 1.27)) hide)
+    )
+    (property "Datasheet" "" (at 121.92 38.1 0)
+      (effects (font (size 1.27 1.27)) hide)
+    )
+    (pin "1")
+    (instances
+      (project "PCB_evenwicht"
+        (path "/1568d5f0-bcdb-494d-bbf5-b93d65138b4f"
+          (reference "#PWR033") (unit 1)
+        )
+        (path "/1568d5f0-bcdb-494d-bbf5-b93d65138b4f/de18e6c3-6c35-4eb3-86ab-f4d9b06c1c30"
+          (reference "#PWR053") (unit 1)
+        )
+      )
+      (project "a4988"
+        (path "/33277f75-9959-42fa-8608-f9642a2ecd81"
+          (reference "#PWR?") (unit 1)
+        )
+      )
+    )
+  )
   (symbol (lib_id "Device:C") (at 113.03 57.15 0) (unit 1)
     (in_bom yes) (on_board yes) (dnp no) (fields_autoplaced)
@@
       (effects (font (size 1.27 1.27)) (justify left))
     )
-    (property "Value" "100uF" (at 111.76 43.815 0)
-      (effects (font (size 1.27 1.27)) (justify left))
-    )
+    (property "Value" "100nF" (at 111.76 43.815 0)
+      (effects (font (size 1.27 1.27)) (justify left))
+    )

Commit message: update pcb
Parts:
- C10, C17, C5, C6, C7, C8, C9: footprint (none) -> Capacitor_SMD:C_0603_1608Metric_Pad1.08x0.95mm_HandSolder
- R10, R11, R8, R9: footprint (none) -> Resistor_SMD:R_0805_2012Metric_Pad1.20x1.40mm_HandSolder
Changed lines of the file:
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@@
       (effects (font (size 1.27 1.27)))
     )
-    (property "Footprint" "" (at 132.08 52.3748 0)
+    (property "Footprint" "Capacitor_SMD:C_0603_1608Metric_Pad1.08x0.95mm_HandSolder" (at 132.08 52.3748 0)
       (effects (font (size 1.27 1.27)) hide)
     )
@@
       (effects (font (size 1.27 1.27)) (justify left))
     )
-    (property "Footprint" "" (at 136.8552 67.31 0)
+    (property "Footprint" "Capacitor_SMD:C_0603_1608Metric_Pad1.08x0.95mm_HandSolder" (at 136.8552 67.31 0)
       (effects (font (size 1.27 1.27)) hide)
     )
@@
       (effects (font (size 1.27 1.27)) (justify left))
     )
-    (property "Footprint" "" (at 122.8852 45.72 0)
+    (property "Footprint" "Capacitor_SMD:C_0603_1608Metric_Pad1.08x0.95mm_HandSolder" (at 122.8852 45.72 0)
       (effects (font (size 1.27 1.27)) hide)
     )
@@
       (effects (font (size 1.27 1.27)))
     )
-    (property "Footprint" "" (at 78.74 37.7952 0)
+    (property "Footprint" "Capacitor_SMD:C_0603_1608Metric_Pad1.08x0.95mm_HandSolder" (at 78.74 37.7952 0)
       (effects (font (size 1.27 1.27)) hide)
     )
@@
       (effects (font (size 1.27 1.27)) (justify right))
     )
-    (property "Footprint" "" (at 62.738 43.18 90)
+    (property "Footprint" "Resistor_SMD:R_0805_2012Metric_Pad1.20x1.40mm_HandSolder" (at 62.738 43.18 90)
       (effects (font (size 1.27 1.27)) hide)
     )
@@
       (effects (font (size 1.27 1.27)) (justify left))
     )
-    (property "Footprint" "" (at 103.8352 105.41 0)
+    (property "Footprint" "Capacitor_SMD:C_0603_1608Metric_Pad1.08x0.95mm_HandSolder" (at 103.8352 105.41 0)
       (effects (font (size 1.27 1.27)) hide)
     )
@@
       (effects (font (size 1.27 1.27)))
     )
-    (property "Footprint" "" (at 115.062 96.52 90)
+    (property "Footprint" "Resistor_SMD:R_0805_2012Metric_Pad1.20x1.40mm_HandSolder" (at 115.062 96.52 90)
       (effects (font (size 1.27 1.27)) hide)
     )
@@
       (effects (font (size 1.27 1.27)) (justify left))
     )
-    (property "Footprint" "" (at 113.9952 60.96 0)
+    (property "Footprint" "Capacitor_SMD:C_0603_1608Metric_Pad1.08x0.95mm_HandSolder" (at 113.9952 60.96 0)
       (effects (font (size 1.27 1.27)) hide)
     )
@@
       (effects (font (size 1.27 1.27)) (justify left))
     )
-    (property "Footprint" "" (at 108.9152 45.72 0)
+    (property "Footprint" "Capacitor_SMD:C_0603_1608Metric_Pad1.08x0.95mm_HandSolder" (at 108.9152 45.72 0)
       (effects (font (size 1.27 1.27)) hide)
     )
@@
       (effects (font (size 1.27 1.27)))
     )
-    (property "Footprint" "" (at 60.96 56.388 90)
+    (property "Footprint" "Resistor_SMD:R_0805_2012Metric_Pad1.20x1.40mm_HandSolder" (at 60.96 56.388 90)
       (effects (font (size 1.27 1.27)) hide)
     )
@@
       (effects (font (size 1.27 1.27)))
     )
-    (property "Footprint" "" (at 120.142 96.52 90)
-      (effects (font (size 1.27 1.27)) hide)
-    )
+    (property "Footprint" "Resistor_SMD:R_0805_2012Metric_Pad1.20x1.40mm_HandSolder" (at 120.142 96.52 90)
+      (effects (font (size 1.27 1.27)) hide)
+    )

Commit message: Update_Update
PCB eens snel geroute
Parts:
- C10, C5, C6, C7, C8, C9: footprint Capacitor_SMD:C_0603_1608Metric_Pad1.08x0.95mm_HandSolder -> Capacitor_SMD:C_0805_2012Metric_Pad1.18x1.45mm_HandSolder
- C17: footprint Capacitor_SMD:C_0603_1608Metric_Pad1.08x0.95mm_HandSolder -> Capacitor_SMD:C_1206_3216Metric_Pad1.33x1.80mm_HandSolder
Connections:
- net VDD is gone; now on net +3.3V: C10.1, IC1.15 (VDD)
Changed lines of the file:
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@@
-    )
-  )
-  (global_label "VDD" (shape input) (at 160.02 59.69 0) (fields_autoplaced)
-    (effects (font (size 1.27 1.27)) (justify left))
-    (property "Intersheetrefs" "${INTERSHEET_REFS}" (at 166.5544 59.69 0)
-      (effects (font (size 1.27 1.27)) (justify left) hide)
     )
   )
@@
       (effects (font (size 1.27 1.27)))
     )
-    (property "Footprint" "Capacitor_SMD:C_0603_1608Metric_Pad1.08x0.95mm_HandSolder" (at 132.08 52.3748 0)
+    (property "Footprint" "Capacitor_SMD:C_0805_2012Metric_Pad1.18x1.45mm_HandSolder" (at 132.08 52.3748 0)
       (effects (font (size 1.27 1.27)) hide)
     )
@@
       (effects (font (size 1.27 1.27)) (justify left))
     )
-    (property "Footprint" "Capacitor_SMD:C_0603_1608Metric_Pad1.08x0.95mm_HandSolder" (at 136.8552 67.31 0)
+    (property "Footprint" "Capacitor_SMD:C_0805_2012Metric_Pad1.18x1.45mm_HandSolder" (at 136.8552 67.31 0)
       (effects (font (size 1.27 1.27)) hide)
     )
@@
       (effects (font (size 1.27 1.27)) (justify left))
     )
-    (property "Footprint" "Capacitor_SMD:C_0603_1608Metric_Pad1.08x0.95mm_HandSolder" (at 122.8852 45.72 0)
+    (property "Footprint" "Capacitor_SMD:C_1206_3216Metric_Pad1.33x1.80mm_HandSolder" (at 122.8852 45.72 0)
       (effects (font (size 1.27 1.27)) hide)
     )
@@
       (effects (font (size 1.27 1.27)))
     )
-    (property "Footprint" "Capacitor_SMD:C_0603_1608Metric_Pad1.08x0.95mm_HandSolder" (at 78.74 37.7952 0)
+    (property "Footprint" "Capacitor_SMD:C_0805_2012Metric_Pad1.18x1.45mm_HandSolder" (at 78.74 37.7952 0)
       (effects (font (size 1.27 1.27)) hide)
     )
@@
       (effects (font (size 1.27 1.27)) (justify left))
     )
-    (property "Footprint" "Capacitor_SMD:C_0603_1608Metric_Pad1.08x0.95mm_HandSolder" (at 103.8352 105.41 0)
+    (property "Footprint" "Capacitor_SMD:C_0805_2012Metric_Pad1.18x1.45mm_HandSolder" (at 103.8352 105.41 0)
       (effects (font (size 1.27 1.27)) hide)
     )
@@
       (effects (font (size 1.27 1.27)) (justify left))
     )
-    (property "Footprint" "Capacitor_SMD:C_0603_1608Metric_Pad1.08x0.95mm_HandSolder" (at 113.9952 60.96 0)
+    (property "Footprint" "Capacitor_SMD:C_0805_2012Metric_Pad1.18x1.45mm_HandSolder" (at 113.9952 60.96 0)
       (effects (font (size 1.27 1.27)) hide)
     )
@@
       (effects (font (size 1.27 1.27)) (justify left))
     )
-    (property "Footprint" "Capacitor_SMD:C_0603_1608Metric_Pad1.08x0.95mm_HandSolder" (at 108.9152 45.72 0)
+    (property "Footprint" "Capacitor_SMD:C_0805_2012Metric_Pad1.18x1.45mm_HandSolder" (at 108.9152 45.72 0)
       (effects (font (size 1.27 1.27)) hide)
     )
@@
         )
       )
+    )
+  )
+  (symbol (lib_id "power:+3.3V") (at 160.02 59.69 0) (unit 1)
+    (in_bom yes) (on_board yes) (dnp no) (fields_autoplaced)
+    (property "Reference" "#PWR055" (at 160.02 63.5 0)
+      (effects (font (size 1.27 1.27)) hide)
+    )
+    (property "Value" "+3.3V" (at 160.02 55.88 0)
+      (effects (font (size 1.27 1.27)))
+    )
+    (property "Footprint" "" (at 160.02 59.69 0)
+      (effects (font (size 1.27 1.27)) hide)
+    )
+    (property "Datasheet" "" (at 160.02 59.69 0)
+      (effects (font (size 1.27 1.27)) hide)
+    )
+    (pin "1")
+    (instances
+      (project "PCB_evenwicht"
+        (path "/1568d5f0-bcdb-494d-bbf5-b93d65138b4f/de18e6c3-6c35-4eb3-86ab-f4d9b06c1c30"
+          (reference "#PWR055") (unit 1)
+        )
+      )

Commit message: fdq
Parts:
- added RV1: R_Potentiometer, Potentiometer_THT:Potentiometer_Bourns_3386P_Vertical, symbol Device:R_Potentiometer
Connections:
- net !RESET is gone; now on net GND: IC1.12 (~{RESET})
- net !SLEEP is gone; now on net GND: IC1.14 (~{SLEEP}), R8.1
- net +3.3V: now also RV1.1
- net GND: now also RV1.3
- net REF1: no longer names the net of IC1.17 (REF)
- net REF1: now also RV1.2
Changed lines of the file:
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@@
-    )
-  )
-  (global_label "!RESET" (shape input) (at 64.77 67.31 180) (fields_autoplaced)
-    (effects (font (size 1.27 1.27)) (justify right))
-    (property "Intersheetrefs" "${INTERSHEET_REFS}" (at 55.5143 67.31 0)
-      (effects (font (size 1.27 1.27)) (justify right) hide)
     )
   )
@@
     )
   )
-  (global_label "!SLEEP" (shape input) (at 54.61 49.53 180) (fields_autoplaced)
-    (effects (font (size 1.27 1.27)) (justify right))
-    (property "Intersheetrefs" "${INTERSHEET_REFS}" (at 45.2938 49.53 0)
-      (effects (font (size 1.27 1.27)) (justify right) hide)
-    )
-  )
   (global_label "GPIO19" (shape input) (at 64.77 62.23 180) (fields_autoplaced)
     (effects (font (size 1.27 1.27)) (justify right))
@@
     )
   )
-  (global_label "REF1" (shape input) (at 50.8 87.63 180) (fields_autoplaced)
-    (effects (font (size 1.27 1.27)) (justify right))
-    (property "Intersheetrefs" "${INTERSHEET_REFS}" (at 43.1771 87.63 0)
-      (effects (font (size 1.27 1.27)) (justify right) hide)
-    )
-  )
   (global_label "Vmot" (shape input) (at 137.16 45.72 0) (fields_autoplaced)
     (effects (font (size 1.27 1.27)) (justify left))
@@
     )
   )
+  (symbol (lib_id "power:GND") (at 64.77 67.31 270) (unit 1)
+    (in_bom yes) (on_board yes) (dnp no) (fields_autoplaced)
+    (property "Reference" "#PWR062" (at 58.42 67.31 0)
+      (effects (font (size 1.27 1.27)) hide)
+    )
+    (property "Value" "GND" (at 60.96 67.945 90)
+      (effects (font (size 1.27 1.27)) (justify right))
+    )
+    (property "Footprint" "" (at 64.77 67.31 0)
+      (effects (font (size 1.27 1.27)) hide)
+    )
+    (property "Datasheet" "" (at 64.77 67.31 0)
+      (effects (font (size 1.27 1.27)) hide)
+    )
+    (pin "1")
+    (instances
+      (project "PCB_evenwicht"
+        (path "/1568d5f0-bcdb-494d-bbf5-b93d65138b4f/de18e6c3-6c35-4eb3-86ab-f4d9b06c1c30"
+          (reference "#PWR062") (unit 1)
+        )
+      )
+    )
+  )
+  (symbol (lib_id "power:GND") (at 54.61 49.53 270) (unit 1)
+    (in_bom yes) (on_board yes) (dnp no) (fields_autoplaced)
+    (property "Reference" "#PWR061" (at 48.26 49.53 0)
+      (effects (font (size 1.27 1.27)) hide)
+    )
+    (property "Value" "GND" (at 50.8 50.165 90)
+      (effects (font (size 1.27 1.27)) (justify right))
+    )
+    (property "Footprint" "" (at 54.61 49.53 0)
+      (effects (font (size 1.27 1.27)) hide)
+    )
+    (property "Datasheet" "" (at 54.61 49.53 0)
+      (effects (font (size 1.27 1.27)) hide)
+    )
+    (pin "1")
+    (instances
+      (project "PCB_evenwicht"
+        (path "/1568d5f0-bcdb-494d-bbf5-b93d65138b4f/de18e6c3-6c35-4eb3-86ab-f4d9b06c1c30"
+          (reference "#PWR061") (unit 1)
+        )
+      )
+    )
+  )
   (symbol (lib_id "Connector:Conn_01x04_Pin") (at 121.92 78.74 180) (unit 1)
     (in_bom yes) (on_board yes) (dnp no) (fields_autoplaced)
@@
     )
   )
+  (symbol (lib_id "Device:R_Potentiometer") (at 46.99 87.63 0) (unit 1)
+    (in_bom yes) (on_board yes) (dnp no) (fields_autoplaced)
+    (property "Reference" "RV1" (at 44.45 86.995 0)
+      (effects (font (size 1.27 1.27)) (justify right))
+    )
+    (property "Value" "R_Potentiometer" (at 44.45 89.535 0)
+      (effects (font (size 1.27 1.27)) (justify right))
+    )
+    (property "Footprint" "Potentiometer_THT:Potentiometer_Bourns_3386P_Vertical" (at 46.99 87.63 0)
+      (effects (font (size 1.27 1.27)) hide)
+    )
+    (property "Datasheet" "~" (at 46.99 87.63 0)
+      (effects (font (size 1.27 1.27)) hide)
+    )
+    (pin "1")
+    (pin "2")
+    (pin "3")
+    (instances
+      (project "PCB_evenwicht"
+        (path "/1568d5f0-bcdb-494d-bbf5-b93d65138b4f/de18e6c3-6c35-4eb3-86ab-f4d9b06c1c30"
+          (reference "RV1") (unit 1)
+        )
+      )
+    )
+  )
   (symbol (lib_id "Device:C") (at 102.87 101.6 0) (unit 1)
     (in_bom yes) (on_board yes) (dnp no) (fields_autoplaced)
@@
         (path "/33277f75-9959-42fa-8608-f9642a2ecd81"
           (reference "#PWR?") (unit 1)
+        )
+      )
+    )
+  )
+  (symbol (lib_id "power:+3.3V") (at 46.99 83.82 0) (unit 1)
+    (in_bom yes) (on_board yes) (dnp no) (fields_autoplaced)
+    (property "Reference" "#PWR057" (at 46.99 87.63 0)
+      (effects (font (size 1.27 1.27)) hide)
+    )
+    (property "Value" "+3.3V" (at 46.99 80.01 0)
+      (effects (font (size 1.27 1.27)))
+    )
+    (property "Footprint" "" (at 46.99 83.82 0)
+      (effects (font (size 1.27 1.27)) hide)
+    )
+    (property "Datasheet" "" (at 46.99 83.82 0)
+      (effects (font (size 1.27 1.27)) hide)
+    )
+    (pin "1")
+    (instances
+      (project "PCB_evenwicht"
+        (path "/1568d5f0-bcdb-494d-bbf5-b93d65138b4f/de18e6c3-6c35-4eb3-86ab-f4d9b06c1c30"
+          (reference "#PWR057") (unit 1)
         )
       )
@@
         )
       )
+    )
+  )
+  (symbol (lib_id "power:GND") (at 46.99 91.44 0) (unit 1)
+    (in_bom yes) (on_board yes) (dnp no) (fields_autoplaced)
+    (property "Reference" "#PWR058" (at 46.99 97.79 0)
+      (effects (font (size 1.27 1.27)) hide)
+    )
+    (property "Value" "GND" (at 46.99 96.52 0)
+      (effects (font (size 1.27 1.27)))
+    )
+    (property "Footprint" "" (at 46.99 91.44 0)
+      (effects (font (size 1.27 1.27)) hide)
+    )
+    (property "Datasheet" "" (at 46.99 91.44 0)
+      (effects (font (size 1.27 1.27)) hide)
+    )
+    (pin "1")
+    (instances
+      (project "PCB_evenwicht"
+        (path "/1568d5f0-bcdb-494d-bbf5-b93d65138b4f/de18e6c3-6c35-4eb3-86ab-f4d9b06c1c30"
+          (reference "#PWR058") (unit 1)
+        )
+      )
