File: PCB_evenwicht/a4988_1.kicad_sch (KiCad schematic)
At the start: 14 parts, among them IC1 A4988SETTR-T, J4 Conn_01x04_Pin

Commit message: fdqjmlk
Parts:
- removed R8: 100K, Resistor_SMD:R_0805_2012Metric_Pad1.20x1.40mm_HandSolder, symbol Device:R
- added C20: 47uF, Capacitor_SMD:CP_Elec_6.3x5.9, symbol Device:C_Polarized
Connections:
- net +3.3V: now also IC1.14 (~{SLEEP})
- net GND: now also IC1.29 (EP), C20.2; no longer IC1.14 (~{SLEEP})
- net Vmot: now also C20.1
- no-connect marks 4 -> 3
Changed lines of the file:
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@@
   (junction (at 102.87 105.41) (diameter 0) (color 0 0 0 0)
   )
-  (junction (at 60.96 49.53) (diameter 0) (color 0 0 0 0)
-  )
   (junction (at 107.95 52.07) (diameter 0) (color 0 0 0 0)
   )
+  (junction (at 133.35 45.72) (diameter 0) (color 0 0 0 0)
+  )
   (junction (at 113.03 53.34) (diameter 0) (color 0 0 0 0)
   )
@@
   (junction (at 121.92 45.72) (diameter 0) (color 0 0 0 0)
   )
-  (no_connect (at 64.77 97.79))
   (no_connect (at 80.01 107.95))
   (no_connect (at 85.09 107.95))
@@
     (stroke (width 0) (type default))
   )
-  (wire (pts (xy 60.96 36.83) (xy 60.96 39.37))
-    (stroke (width 0) (type default))
-  )
   (wire (pts (xy 107.95 52.07) (xy 107.95 53.34))
     (stroke (width 0) (type default))
@@
     (stroke (width 0) (type default))
   )
-  (wire (pts (xy 60.96 46.99) (xy 60.96 49.53))
+  (wire (pts (xy 55.88 49.53) (xy 64.77 49.53))
     (stroke (width 0) (type default))
   )
@@
     (stroke (width 0) (type default))
   )
-  (wire (pts (xy 121.92 45.72) (xy 137.16 45.72))
+  (wire (pts (xy 121.92 45.72) (xy 133.35 45.72))
     (stroke (width 0) (type default))
   )
@@
     (stroke (width 0) (type default))
   )
-  (wire (pts (xy 54.61 49.53) (xy 60.96 49.53))
+  (wire (pts (xy 133.35 45.72) (xy 142.24 45.72))
     (stroke (width 0) (type default))
   )
@@
   )
   (wire (pts (xy 85.09 39.37) (xy 86.36 39.37))
-    (stroke (width 0) (type default))
-  )
-  (wire (pts (xy 60.96 49.53) (xy 64.77 49.53))
     (stroke (width 0) (type default))
   )
@@
     )
   )
-  (global_label "Vmot" (shape input) (at 137.16 45.72 0) (fields_autoplaced)
+  (global_label "Vmot" (shape input) (at 142.24 45.72 0) (fields_autoplaced)
     (effects (font (size 1.27 1.27)) (justify left))
-    (property "Intersheetrefs" "${INTERSHEET_REFS}" (at 144.7224 45.72 0)
+    (property "Intersheetrefs" "${INTERSHEET_REFS}" (at 149.8024 45.72 0)
       (effects (font (size 1.27 1.27)) (justify left) hide)
     )
@@
     )
   )
-  (symbol (lib_id "power:GND") (at 54.61 49.53 270) (unit 1)
-    (in_bom yes) (on_board yes) (dnp no) (fields_autoplaced)
-    (property "Reference" "#PWR061" (at 48.26 49.53 0)
-      (effects (font (size 1.27 1.27)) hide)
-    )
-    (property "Value" "GND" (at 50.8 50.165 90)
-      (effects (font (size 1.27 1.27)) (justify right))
-    )
-    (property "Footprint" "" (at 54.61 49.53 0)
-      (effects (font (size 1.27 1.27)) hide)
-    )
-    (property "Datasheet" "" (at 54.61 49.53 0)
-      (effects (font (size 1.27 1.27)) hide)
-    )
-    (pin "1")
-    (instances
-      (project "PCB_evenwicht"
-        (path "/1568d5f0-bcdb-494d-bbf5-b93d65138b4f/de18e6c3-6c35-4eb3-86ab-f4d9b06c1c30"
-          (reference "#PWR061") (unit 1)
-        )
-      )
-    )
-  )
   (symbol (lib_id "Connector:Conn_01x04_Pin") (at 121.92 78.74 180) (unit 1)
     (in_bom yes) (on_board yes) (dnp no) (fields_autoplaced)
@@
         (path "/1568d5f0-bcdb-494d-bbf5-b93d65138b4f/de18e6c3-6c35-4eb3-86ab-f4d9b06c1c30"
           (reference "J4") (unit 1)
+        )
+      )
+    )
+  )
+  (symbol (lib_id "power:GND") (at 133.35 38.1 180) (unit 1)
+    (in_bom yes) (on_board yes) (dnp no) (fields_autoplaced)
+    (property "Reference" "#PWR066" (at 133.35 31.75 0)
+      (effects (font (size 1.27 1.27)) hide)
+    )
+    (property "Value" "GND" (at 133.35 34.29 0)
+      (effects (font (size 1.27 1.27)))
+    )
+    (property "Footprint" "" (at 133.35 38.1 0)
+      (effects (font (size 1.27 1.27)) hide)
+    )
+    (property "Datasheet" "" (at 133.35 38.1 0)
+      (effects (font (size 1.27 1.27)) hide)
+    )
+    (pin "1")
+    (instances
+      (project "PCB_evenwicht"
+        (path "/1568d5f0-bcdb-494d-bbf5-b93d65138b4f/de18e6c3-6c35-4eb3-86ab-f4d9b06c1c30"
+          (reference "#PWR066") (unit 1)
         )
       )
@@
     )
   )
+  (symbol (lib_id "power:+3.3V") (at 55.88 49.53 0) (unit 1)
+    (in_bom yes) (on_board yes) (dnp no) (fields_autoplaced)
+    (property "Reference" "#PWR067" (at 55.88 53.34 0)
+      (effects (font (size 1.27 1.27)) hide)
+    )
+    (property "Value" "+3.3V" (at 55.88 45.72 0)
+      (effects (font (size 1.27 1.27)))
+    )
+    (property "Footprint" "" (at 55.88 49.53 0)
+      (effects (font (size 1.27 1.27)) hide)
+    )
+    (property "Datasheet" "" (at 55.88 49.53 0)
+      (effects (font (size 1.27 1.27)) hide)
+    )
+    (pin "1")
+    (instances
+      (project "PCB_evenwicht"
+        (path "/1568d5f0-bcdb-494d-bbf5-b93d65138b4f/de18e6c3-6c35-4eb3-86ab-f4d9b06c1c30"
+          (reference "#PWR067") (unit 1)
+        )
+      )
+    )
+  )
+  (symbol (lib_id "power:GND") (at 64.77 97.79 270) (unit 1)
+    (in_bom yes) (on_board yes) (dnp no) (fields_autoplaced)
+    (property "Reference" "#PWR061" (at 58.42 97.79 0)
+      (effects (font (size 1.27 1.27)) hide)
+    )
+    (property "Value" "GND" (at 60.96 98.425 90)
+      (effects (font (size 1.27 1.27)) (justify right))
+    )
+    (property "Footprint" "" (at 64.77 97.79 0)
+      (effects (font (size 1.27 1.27)) hide)
+    )
+    (property "Datasheet" "" (at 64.77 97.79 0)
+      (effects (font (size 1.27 1.27)) hide)
+    )
+    (pin "1")
+    (instances
+      (project "PCB_evenwicht"
+        (path "/1568d5f0-bcdb-494d-bbf5-b93d65138b4f/de18e6c3-6c35-4eb3-86ab-f4d9b06c1c30"
+          (reference "#PWR061") (unit 1)
+        )
+      )
+    )
+  )
   (symbol (lib_id "power:GND") (at 107.95 38.1 180) (unit 1)
     (in_bom yes) (on_board yes) (dnp no) (fields_autoplaced)
@@
         (path "/33277f75-9959-42fa-8608-f9642a2ecd81"
           (reference "C?") (unit 1)
-        )
-      )
-    )
-  )
-  (symbol (lib_id "Device:R") (at 60.96 43.18 180) (unit 1)
-    (in_bom yes) (on_board yes) (dnp no)
-    (property "Reference" "R8" (at 63.5 42.545 0)
-      (effects (font (size 1.27 1.27)) (justify right))
-    )
-    (property "Value" "100K" (at 63.5 44.45 0)
-      (effects (font (size 1.27 1.27)) (justify right))
-    )
-    (property "Footprint" "Resistor_SMD:R_0805_2012Metric_Pad1.20x1.40mm_HandSolder" (at 62.738 43.18 90)
-      (effects (font (size 1.27 1.27)) hide)
-    )
-    (property "Datasheet" "~" (at 60.96 43.18 0)
-      (effects (font (size 1.27 1.27)) hide)
-    )
-    (pin "1")
-    (pin "2")
-    (instances
-      (project "PCB_evenwicht"
-        (path "/1568d5f0-bcdb-494d-bbf5-b93d65138b4f"
-          (reference "R8") (unit 1)
-        )
-        (path "/1568d5f0-bcdb-494d-bbf5-b93d65138b4f/de18e6c3-6c35-4eb3-86ab-f4d9b06c1c30"
-          (reference "R8") (unit 1)
-        )
-      )
-      (project "a4988"
-        (path "/33277f75-9959-42fa-8608-f9642a2ecd81"
-          (reference "R?") (unit 1)
         )
       )
@@
     )
   )
-  (symbol (lib_id "power:+3.3V") (at 60.96 36.83 0) (unit 1)
-    (in_bom yes) (on_board yes) (dnp no) (fields_autoplaced)
-    (property "Reference" "#PWR028" (at 60.96 40.64 0)
-      (effects (font (size 1.27 1.27)) hide)
-    )
-    (property "Value" "+3.3V" (at 60.96 33.02 0)
-      (effects (font (size 1.27 1.27)))
-    )
-    (property "Footprint" "" (at 60.96 36.83 0)
-      (effects (font (size 1.27 1.27)) hide)
-    )
-    (property "Datasheet" "" (at 60.96 36.83 0)
-      (effects (font (size 1.27 1.27)) hide)
-    )
-    (pin "1")
-    (instances
-      (project "PCB_evenwicht"
-        (path "/1568d5f0-bcdb-494d-bbf5-b93d65138b4f"
-          (reference "#PWR028") (unit 1)
-        )
-        (path "/1568d5f0-bcdb-494d-bbf5-b93d65138b4f/de18e6c3-6c35-4eb3-86ab-f4d9b06c1c30"
-          (reference "#PWR028") (unit 1)
-        )
-      )
+  (symbol (lib_id "Device:C_Polarized") (at 133.35 41.91 180) (unit 1)
+    (in_bom yes) (on_board yes) (dnp no)
+    (property "Reference" "C20" (at 137.16 40.64 0)
+      (effects (font (size 1.27 1.27)) (justify right))
+    )
+    (property "Value" "47uF" (at 137.16 43.18 0)
+      (effects (font (size 1.27 1.27)) (justify right))
+    )
+    (property "Footprint" "Capacitor_SMD:CP_Elec_6.3x5.9" (at 132.3848 38.1 0)
+      (effects (font (size 1.27 1.27)) hide)
+    )
+    (property "Datasheet" "~" (at 133.35 41.91 0)
+      (effects (font (size 1.27 1.27)) hide)
+    )
+    (pin "1")
+    (pin "2")
+    (instances
+      (project "PCB_evenwicht"
+        (path "/1568d5f0-bcdb-494d-bbf5-b93d65138b4f/de18e6c3-6c35-4eb3-86ab-f4d9b06c1c30"
+          (reference "C20") (unit 1)
+        )
+      )

Commit message: goed
Parts:
- C17: footprint Capacitor_SMD:C_1206_3216Metric_Pad1.33x1.80mm_HandSolder -> Capacitor_SMD:C_0805_2012Metric_Pad1.18x1.45mm_HandSolder
Connections:
- net +3.3V: now also IC1.12 (~{RESET})
- net GND: no longer IC1.12 (~{RESET})
Changed lines of the file:
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@@
+    (stroke (width 0) (type default))
+  )
+  (wire (pts (xy 52.07 67.31) (xy 64.77 67.31))
     (stroke (width 0) (type default))
   )
@@
     )
   )
-  (symbol (lib_id "power:GND") (at 64.77 67.31 270) (unit 1)
-    (in_bom yes) (on_board yes) (dnp no) (fields_autoplaced)
-    (property "Reference" "#PWR062" (at 58.42 67.31 0)
-      (effects (font (size 1.27 1.27)) hide)
-    )
-    (property "Value" "GND" (at 60.96 67.945 90)
-      (effects (font (size 1.27 1.27)) (justify right))
-    )
-    (property "Footprint" "" (at 64.77 67.31 0)
-      (effects (font (size 1.27 1.27)) hide)
-    )
-    (property "Datasheet" "" (at 64.77 67.31 0)
-      (effects (font (size 1.27 1.27)) hide)
-    )
-    (pin "1")
-    (instances
-      (project "PCB_evenwicht"
+  (symbol (lib_id "power:+3.3V") (at 52.07 67.31 0) (unit 1)
+    (in_bom yes) (on_board yes) (dnp no) (fields_autoplaced)
+    (property "Reference" "#PWR028" (at 52.07 71.12 0)
+      (effects (font (size 1.27 1.27)) hide)
+    )
+    (property "Value" "+3.3V" (at 52.07 63.5 0)
+      (effects (font (size 1.27 1.27)))
+    )
+    (property "Footprint" "" (at 52.07 67.31 0)
+      (effects (font (size 1.27 1.27)) hide)
+    )
+    (property "Datasheet" "" (at 52.07 67.31 0)
+      (effects (font (size 1.27 1.27)) hide)
+    )
+    (pin "1")
+    (instances
+      (project "PCB_evenwicht"
+        (path "/1568d5f0-bcdb-494d-bbf5-b93d65138b4f/0fee5d6f-552e-4af4-870f-decaeb093c62"
+          (reference "#PWR028") (unit 1)
+        )
         (path "/1568d5f0-bcdb-494d-bbf5-b93d65138b4f/de18e6c3-6c35-4eb3-86ab-f4d9b06c1c30"
           (reference "#PWR062") (unit 1)
@@
       (effects (font (size 1.27 1.27)) (justify left))
     )
-    (property "Footprint" "Capacitor_SMD:C_1206_3216Metric_Pad1.33x1.80mm_HandSolder" (at 122.8852 45.72 0)
-      (effects (font (size 1.27 1.27)) hide)
-    )
+    (property "Footprint" "Capacitor_SMD:C_0805_2012Metric_Pad1.18x1.45mm_HandSolder" (at 122.8852 45.72 0)
+      (effects (font (size 1.27 1.27)) hide)
+    )
