File: PCB_evenwicht/a4988_2.kicad_sch (KiCad schematic)
At the start: 12 parts, among them IC1 A4988SETTR-T, J4 Conn_01x04_Pin

Commit message: update
Connections:
- no-connect marks 3 -> 4
Changed lines of the file:
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@@
   (no_connect (at 78.74 105.41))
   (no_connect (at 76.2 105.41))
+  (no_connect (at 58.42 95.25))
   (no_connect (at 73.66 105.41))
   (wire (pts (xy 107.95 67.31) (xy 107.95 71.12))

Commit message: update pcb-design
Parts:
- added C17: 4.7uF, symbol Device:C
- C7, C9: value 100uF -> 100nF
Connections:
- net GND: now also C17.1
- net Vmot: now also C17.2
- net GPIO32 renamed GPIO19
- net GPIO33 renamed GPIO18
- net MS1_2 renamed MS1_1
- net MS2_2 renamed MS2_1
- net MS3_2 renamed MS3_1
- net REF2 renamed REF1
Other:
- note removed: "NOG een 4.7uf condensator denk ik ergens plaatsen"

Commit message: update pcb
Parts:
- C10, C17, C5, C6, C7, C8, C9: footprint (none) -> Capacitor_SMD:C_0603_1608Metric_Pad1.08x0.95mm_HandSolder
- R10, R11, R8, R9: footprint (none) -> Resistor_SMD:R_0805_2012Metric_Pad1.20x1.40mm_HandSolder
Changed lines of the file:
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@@
       (effects (font (size 1.27 1.27)))
     )
-    (property "Footprint" "" (at 54.61 55.118 90)
+    (property "Footprint" "Resistor_SMD:R_0805_2012Metric_Pad1.20x1.40mm_HandSolder" (at 54.61 55.118 90)
       (effects (font (size 1.27 1.27)) hide)
     )
@@
       (effects (font (size 1.27 1.27)))
     )
-    (property "Footprint" "" (at 113.792 95.25 90)
+    (property "Footprint" "Resistor_SMD:R_0805_2012Metric_Pad1.20x1.40mm_HandSolder" (at 113.792 95.25 90)
       (effects (font (size 1.27 1.27)) hide)
     )
@@
       (effects (font (size 1.27 1.27)))
     )
-    (property "Footprint" "" (at 108.712 95.25 90)
+    (property "Footprint" "Resistor_SMD:R_0805_2012Metric_Pad1.20x1.40mm_HandSolder" (at 108.712 95.25 90)
       (effects (font (size 1.27 1.27)) hide)
     )
@@
       (effects (font (size 1.27 1.27)) (justify right))
     )
-    (property "Footprint" "" (at 56.388 41.91 90)
+    (property "Footprint" "Resistor_SMD:R_0805_2012Metric_Pad1.20x1.40mm_HandSolder" (at 56.388 41.91 90)
       (effects (font (size 1.27 1.27)) hide)
     )
@@
       (effects (font (size 1.27 1.27)) (justify left))
     )
-    (property "Footprint" "" (at 97.4852 104.14 0)
+    (property "Footprint" "Capacitor_SMD:C_0603_1608Metric_Pad1.08x0.95mm_HandSolder" (at 97.4852 104.14 0)
       (effects (font (size 1.27 1.27)) hide)
     )
@@
       (effects (font (size 1.27 1.27)) (justify left))
     )
-    (property "Footprint" "" (at 116.5352 44.45 0)
+    (property "Footprint" "Capacitor_SMD:C_0603_1608Metric_Pad1.08x0.95mm_HandSolder" (at 116.5352 44.45 0)
       (effects (font (size 1.27 1.27)) hide)
     )
@@
       (effects (font (size 1.27 1.27)) (justify left))
     )
-    (property "Footprint" "" (at 102.5652 44.45 0)
+    (property "Footprint" "Capacitor_SMD:C_0603_1608Metric_Pad1.08x0.95mm_HandSolder" (at 102.5652 44.45 0)
       (effects (font (size 1.27 1.27)) hide)
     )
@@
       (effects (font (size 1.27 1.27)))
     )
-    (property "Footprint" "" (at 125.73 51.1048 0)
+    (property "Footprint" "Capacitor_SMD:C_0603_1608Metric_Pad1.08x0.95mm_HandSolder" (at 125.73 51.1048 0)
       (effects (font (size 1.27 1.27)) hide)
     )
@@
       (effects (font (size 1.27 1.27)) (justify left))
     )
-    (property "Footprint" "" (at 130.5052 66.04 0)
+    (property "Footprint" "Capacitor_SMD:C_0603_1608Metric_Pad1.08x0.95mm_HandSolder" (at 130.5052 66.04 0)
       (effects (font (size 1.27 1.27)) hide)
     )
@@
       (effects (font (size 1.27 1.27)) (justify left))
     )
-    (property "Footprint" "" (at 107.6452 59.69 0)
+    (property "Footprint" "Capacitor_SMD:C_0603_1608Metric_Pad1.08x0.95mm_HandSolder" (at 107.6452 59.69 0)
       (effects (font (size 1.27 1.27)) hide)
     )
@@
       (effects (font (size 1.27 1.27)))
     )
-    (property "Footprint" "" (at 72.39 36.5252 0)
-      (effects (font (size 1.27 1.27)) hide)
-    )
+    (property "Footprint" "Capacitor_SMD:C_0603_1608Metric_Pad1.08x0.95mm_HandSolder" (at 72.39 36.5252 0)
+      (effects (font (size 1.27 1.27)) hide)
+    )

Commit message: klj
Connections:
- net GPIO18 renamed A5
- net GPIO19 renamed A4
- net MS1_1 renamed MS1_2
- net MS2_1 renamed MS2_2
- net MS3_1 renamed MS3_2
- net REF1 renamed REF2
Changed lines of the file:
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@@
     (stroke (width 0) (type default))
   )
-  (global_label "GPIO18" (shape input) (at 58.42 58.42 180) (fields_autoplaced)
+  (global_label "A5" (shape input) (at 58.42 58.42 180) (fields_autoplaced)
     (effects (font (size 1.27 1.27)) (justify right))
-    (property "Intersheetrefs" "${INTERSHEET_REFS}" (at 48.6199 58.42 0)
+    (property "Intersheetrefs" "${INTERSHEET_REFS}" (at 53.2161 58.42 0)
       (effects (font (size 1.27 1.27)) (justify right) hide)
     )
   )
-  (global_label "MS1_1" (shape input) (at 58.42 73.66 180) (fields_autoplaced)
+  (global_label "MS1_2" (shape input) (at 58.42 73.66 180) (fields_autoplaced)
     (effects (font (size 1.27 1.27)) (justify right))
     (property "Intersheetrefs" "${INTERSHEET_REFS}" (at 49.4667 73.66 0)
@@
     )
   )
-  (global_label "GPIO19" (shape input) (at 58.42 60.96 180) (fields_autoplaced)
+  (global_label "A4" (shape input) (at 58.42 60.96 180) (fields_autoplaced)
     (effects (font (size 1.27 1.27)) (justify right))
-    (property "Intersheetrefs" "${INTERSHEET_REFS}" (at 48.6199 60.96 0)
+    (property "Intersheetrefs" "${INTERSHEET_REFS}" (at 53.2161 60.96 0)
       (effects (font (size 1.27 1.27)) (justify right) hide)
     )
@@
     )
   )
-  (global_label "MS2_1" (shape input) (at 58.42 71.12 180) (fields_autoplaced)
+  (global_label "MS2_2" (shape input) (at 58.42 71.12 180) (fields_autoplaced)
     (effects (font (size 1.27 1.27)) (justify right))
     (property "Intersheetrefs" "${INTERSHEET_REFS}" (at 49.4667 71.12 0)
@@
     )
   )
-  (global_label "REF1" (shape input) (at 44.45 86.36 180) (fields_autoplaced)
+  (global_label "REF2" (shape input) (at 44.45 86.36 180) (fields_autoplaced)
     (effects (font (size 1.27 1.27)) (justify right))
     (property "Intersheetrefs" "${INTERSHEET_REFS}" (at 36.8271 86.36 0)
@@
     )
   )
-  (global_label "MS3_1" (shape input) (at 58.42 68.58 180) (fields_autoplaced)
+  (global_label "MS3_2" (shape input) (at 58.42 68.58 180) (fields_autoplaced)
     (effects (font (size 1.27 1.27)) (justify right))
     (property "Intersheetrefs" "${INTERSHEET_REFS}" (at 49.4667 68.58 0)

Commit message: Update_Update
PCB eens snel geroute
Parts:
- C10, C5, C6, C7, C8, C9: footprint Capacitor_SMD:C_0603_1608Metric_Pad1.08x0.95mm_HandSolder -> Capacitor_SMD:C_0805_2012Metric_Pad1.18x1.45mm_HandSolder
- C17: footprint Capacitor_SMD:C_0603_1608Metric_Pad1.08x0.95mm_HandSolder -> Capacitor_SMD:C_1206_3216Metric_Pad1.33x1.80mm_HandSolder
Connections:
- net VDD is gone; now on net +3.3V: C10.1, IC1.15 (VDD)
Changed lines of the file:
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@@
-    )
-  )
-  (global_label "VDD" (shape input) (at 153.67 58.42 0) (fields_autoplaced)
-    (effects (font (size 1.27 1.27)) (justify left))
-    (property "Intersheetrefs" "${INTERSHEET_REFS}" (at 160.2044 58.42 0)
-      (effects (font (size 1.27 1.27)) (justify left) hide)
     )
   )
@@
       (effects (font (size 1.27 1.27)) (justify left))
     )
-    (property "Footprint" "Capacitor_SMD:C_0603_1608Metric_Pad1.08x0.95mm_HandSolder" (at 97.4852 104.14 0)
+    (property "Footprint" "Capacitor_SMD:C_0805_2012Metric_Pad1.18x1.45mm_HandSolder" (at 97.4852 104.14 0)
       (effects (font (size 1.27 1.27)) hide)
     )
@@
       (effects (font (size 1.27 1.27)) (justify left))
     )
-    (property "Footprint" "Capacitor_SMD:C_0603_1608Metric_Pad1.08x0.95mm_HandSolder" (at 116.5352 44.45 0)
+    (property "Footprint" "Capacitor_SMD:C_1206_3216Metric_Pad1.33x1.80mm_HandSolder" (at 116.5352 44.45 0)
       (effects (font (size 1.27 1.27)) hide)
     )
@@
       (effects (font (size 1.27 1.27)) (justify left))
     )
-    (property "Footprint" "Capacitor_SMD:C_0603_1608Metric_Pad1.08x0.95mm_HandSolder" (at 102.5652 44.45 0)
+    (property "Footprint" "Capacitor_SMD:C_0805_2012Metric_Pad1.18x1.45mm_HandSolder" (at 102.5652 44.45 0)
       (effects (font (size 1.27 1.27)) hide)
     )
@@
       (effects (font (size 1.27 1.27)))
     )
-    (property "Footprint" "Capacitor_SMD:C_0603_1608Metric_Pad1.08x0.95mm_HandSolder" (at 125.73 51.1048 0)
+    (property "Footprint" "Capacitor_SMD:C_0805_2012Metric_Pad1.18x1.45mm_HandSolder" (at 125.73 51.1048 0)
       (effects (font (size 1.27 1.27)) hide)
     )
@@
         (path "/33277f75-9959-42fa-8608-f9642a2ecd81"
           (reference "C?") (unit 1)
+        )
+      )
+    )
+  )
+  (symbol (lib_id "power:+3.3V") (at 153.67 58.42 0) (unit 1)
+    (in_bom yes) (on_board yes) (dnp no) (fields_autoplaced)
+    (property "Reference" "#PWR056" (at 153.67 62.23 0)
+      (effects (font (size 1.27 1.27)) hide)
+    )
+    (property "Value" "+3.3V" (at 153.67 54.61 0)
+      (effects (font (size 1.27 1.27)))
+    )
+    (property "Footprint" "" (at 153.67 58.42 0)
+      (effects (font (size 1.27 1.27)) hide)
+    )
+    (property "Datasheet" "" (at 153.67 58.42 0)
+      (effects (font (size 1.27 1.27)) hide)
+    )
+    (pin "1")
+    (instances
+      (project "PCB_evenwicht"
+        (path "/1568d5f0-bcdb-494d-bbf5-b93d65138b4f/0fee5d6f-552e-4af4-870f-decaeb093c62"
+          (reference "#PWR056") (unit 1)
         )
       )
@@
       (effects (font (size 1.27 1.27)) (justify left))
     )
-    (property "Footprint" "Capacitor_SMD:C_0603_1608Metric_Pad1.08x0.95mm_HandSolder" (at 130.5052 66.04 0)
+    (property "Footprint" "Capacitor_SMD:C_0805_2012Metric_Pad1.18x1.45mm_HandSolder" (at 130.5052 66.04 0)
       (effects (font (size 1.27 1.27)) hide)
     )
@@
       (effects (font (size 1.27 1.27)) (justify left))
     )
-    (property "Footprint" "Capacitor_SMD:C_0603_1608Metric_Pad1.08x0.95mm_HandSolder" (at 107.6452 59.69 0)
+    (property "Footprint" "Capacitor_SMD:C_0805_2012Metric_Pad1.18x1.45mm_HandSolder" (at 107.6452 59.69 0)
       (effects (font (size 1.27 1.27)) hide)
     )
@@
       (effects (font (size 1.27 1.27)))
     )
-    (property "Footprint" "Capacitor_SMD:C_0603_1608Metric_Pad1.08x0.95mm_HandSolder" (at 72.39 36.5252 0)
-      (effects (font (size 1.27 1.27)) hide)
-    )
+    (property "Footprint" "Capacitor_SMD:C_0805_2012Metric_Pad1.18x1.45mm_HandSolder" (at 72.39 36.5252 0)
+      (effects (font (size 1.27 1.27)) hide)
+    )

Commit message: fdq
Parts:
- added RV2: R_Potentiometer, Potentiometer_THT:Potentiometer_Bourns_3386P_Vertical, symbol Device:R_Potentiometer
Connections:
- net !RESET is gone; now on net GND: IC1.12 (~{RESET})
- net !SLEEP is gone; now on net GND: IC1.14 (~{SLEEP}), R8.1
- net +3.3V: now also RV2.1
- net GND: now also RV2.3
- net REF2: no longer names the net of IC1.17 (REF)
- net REF2: now also RV2.2
Changed lines of the file:
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@@
-    )
-  )
-  (global_label "!SLEEP" (shape input) (at 48.26 48.26 180) (fields_autoplaced)
-    (effects (font (size 1.27 1.27)) (justify right))
-    (property "Intersheetrefs" "${INTERSHEET_REFS}" (at 38.9438 48.26 0)
-      (effects (font (size 1.27 1.27)) (justify right) hide)
     )
   )
@@
     )
   )
-  (global_label "!RESET" (shape input) (at 58.42 66.04 180) (fields_autoplaced)
-    (effects (font (size 1.27 1.27)) (justify right))
-    (property "Intersheetrefs" "${INTERSHEET_REFS}" (at 49.1643 66.04 0)
-      (effects (font (size 1.27 1.27)) (justify right) hide)
-    )
-  )
-  (global_label "REF2" (shape input) (at 44.45 86.36 180) (fields_autoplaced)
-    (effects (font (size 1.27 1.27)) (justify right))
-    (property "Intersheetrefs" "${INTERSHEET_REFS}" (at 36.8271 86.36 0)
-      (effects (font (size 1.27 1.27)) (justify right) hide)
-    )
-  )
   (global_label "MS3_2" (shape input) (at 58.42 68.58 180) (fields_autoplaced)
     (effects (font (size 1.27 1.27)) (justify right))
@@
     )
   )
+  (symbol (lib_id "power:GND") (at 48.26 48.26 270) (unit 1)
+    (in_bom yes) (on_board yes) (dnp no) (fields_autoplaced)
+    (property "Reference" "#PWR063" (at 41.91 48.26 0)
+      (effects (font (size 1.27 1.27)) hide)
+    )
+    (property "Value" "GND" (at 44.45 48.895 90)
+      (effects (font (size 1.27 1.27)) (justify right))
+    )
+    (property "Footprint" "" (at 48.26 48.26 0)
+      (effects (font (size 1.27 1.27)) hide)
+    )
+    (property "Datasheet" "" (at 48.26 48.26 0)
+      (effects (font (size 1.27 1.27)) hide)
+    )
+    (pin "1")
+    (instances
+      (project "PCB_evenwicht"
+        (path "/1568d5f0-bcdb-494d-bbf5-b93d65138b4f/0fee5d6f-552e-4af4-870f-decaeb093c62"
+          (reference "#PWR063") (unit 1)
+        )
+      )
+    )
+  )
+  (symbol (lib_id "Device:R_Potentiometer") (at 40.64 86.36 0) (unit 1)
+    (in_bom yes) (on_board yes) (dnp no) (fields_autoplaced)
+    (property "Reference" "RV2" (at 38.1 85.725 0)
+      (effects (font (size 1.27 1.27)) (justify right))
+    )
+    (property "Value" "R_Potentiometer" (at 38.1 88.265 0)
+      (effects (font (size 1.27 1.27)) (justify right))
+    )
+    (property "Footprint" "Potentiometer_THT:Potentiometer_Bourns_3386P_Vertical" (at 40.64 86.36 0)
+      (effects (font (size 1.27 1.27)) hide)
+    )
+    (property "Datasheet" "~" (at 40.64 86.36 0)
+      (effects (font (size 1.27 1.27)) hide)
+    )
+    (pin "1")
+    (pin "2")
+    (pin "3")
+    (instances
+      (project "PCB_evenwicht"
+        (path "/1568d5f0-bcdb-494d-bbf5-b93d65138b4f/0fee5d6f-552e-4af4-870f-decaeb093c62"
+          (reference "RV2") (unit 1)
+        )
+      )
+    )
+  )
   (symbol (lib_id "power:GND") (at 50.8 53.34 270) (unit 1)
     (in_bom yes) (on_board yes) (dnp no) (fields_autoplaced)
@@
     )
   )
+  (symbol (lib_id "power:GND") (at 40.64 90.17 0) (unit 1)
+    (in_bom yes) (on_board yes) (dnp no) (fields_autoplaced)
+    (property "Reference" "#PWR059" (at 40.64 96.52 0)
+      (effects (font (size 1.27 1.27)) hide)
+    )
+    (property "Value" "GND" (at 40.64 95.25 0)
+      (effects (font (size 1.27 1.27)))
+    )
+    (property "Footprint" "" (at 40.64 90.17 0)
+      (effects (font (size 1.27 1.27)) hide)
+    )
+    (property "Datasheet" "" (at 40.64 90.17 0)
+      (effects (font (size 1.27 1.27)) hide)
+    )
+    (pin "1")
+    (instances
+      (project "PCB_evenwicht"
+        (path "/1568d5f0-bcdb-494d-bbf5-b93d65138b4f/0fee5d6f-552e-4af4-870f-decaeb093c62"
+          (reference "#PWR059") (unit 1)
+        )
+      )
+    )
+  )
   (symbol (lib_id "power:GND") (at 129.54 66.04 0) (unit 1)
     (in_bom yes) (on_board yes) (dnp no) (fields_autoplaced)
@@
         (path "/33277f75-9959-42fa-8608-f9642a2ecd81"
           (reference "#PWR?") (unit 1)
+        )
+      )
+    )
+  )
+  (symbol (lib_id "power:GND") (at 58.42 66.04 270) (unit 1)
+    (in_bom yes) (on_board yes) (dnp no) (fields_autoplaced)
+    (property "Reference" "#PWR064" (at 52.07 66.04 0)
+      (effects (font (size 1.27 1.27)) hide)
+    )
+    (property "Value" "GND" (at 54.61 66.675 90)
+      (effects (font (size 1.27 1.27)) (justify right))
+    )
+    (property "Footprint" "" (at 58.42 66.04 0)
+      (effects (font (size 1.27 1.27)) hide)
+    )
+    (property "Datasheet" "" (at 58.42 66.04 0)
+      (effects (font (size 1.27 1.27)) hide)
+    )
+    (pin "1")
+    (instances
+      (project "PCB_evenwicht"
+        (path "/1568d5f0-bcdb-494d-bbf5-b93d65138b4f/0fee5d6f-552e-4af4-870f-decaeb093c62"
+          (reference "#PWR064") (unit 1)
         )
       )
@@
         )
       )
+    )
+  )
+  (symbol (lib_id "power:+3.3V") (at 40.64 82.55 0) (unit 1)
+    (in_bom yes) (on_board yes) (dnp no) (fields_autoplaced)
+    (property "Reference" "#PWR060" (at 40.64 86.36 0)
+      (effects (font (size 1.27 1.27)) hide)
+    )
+    (property "Value" "+3.3V" (at 40.64 78.74 0)
+      (effects (font (size 1.27 1.27)))
+    )
+    (property "Footprint" "" (at 40.64 82.55 0)
+      (effects (font (size 1.27 1.27)) hide)
+    )
+    (property "Datasheet" "" (at 40.64 82.55 0)
+      (effects (font (size 1.27 1.27)) hide)
+    )
+    (pin "1")
+    (instances
+      (project "PCB_evenwicht"
+        (path "/1568d5f0-bcdb-494d-bbf5-b93d65138b4f/0fee5d6f-552e-4af4-870f-decaeb093c62"
+          (reference "#PWR060") (unit 1)
+        )
+      )
