File: PCB_evenwicht/a4988_2.kicad_sch (KiCad schematic)
At the start: 14 parts, among them IC1 A4988SETTR-T, J4 Conn_01x04_Pin

Commit message: fdqjmlk
Parts:
- removed R8: 100K, Resistor_SMD:R_0805_2012Metric_Pad1.20x1.40mm_HandSolder, symbol Device:R
- added C19: 47uF, Capacitor_SMD:CP_Elec_6.3x5.9, symbol Device:C_Polarized
Connections:
- net +3.3V: now also IC1.14 (~{SLEEP})
- net GND: now also IC1.29 (EP), C19.2; no longer IC1.14 (~{SLEEP})
- net Vmot: now also C19.1
- no-connect marks 4 -> 3
Changed lines of the file:
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@@
   (junction (at 101.6 48.26) (diameter 0) (color 0 0 0 0)
   )
-  (junction (at 54.61 48.26) (diameter 0) (color 0 0 0 0)
+  (junction (at 127 44.45) (diameter 0) (color 0 0 0 0)
   )
   (junction (at 106.68 52.07) (diameter 0) (color 0 0 0 0)
@@
   (no_connect (at 76.2 106.68))
   (no_connect (at 78.74 106.68))
-  (no_connect (at 58.42 96.52))
   (no_connect (at 73.66 106.68))
-  (wire (pts (xy 48.26 48.26) (xy 54.61 48.26))
+  (wire (pts (xy 48.26 48.26) (xy 58.42 48.26))
     (stroke (width 0) (type default))
   )
@@
     (stroke (width 0) (type default))
   )
-  (wire (pts (xy 115.57 44.45) (xy 130.81 44.45))
+  (wire (pts (xy 115.57 44.45) (xy 127 44.45))
     (stroke (width 0) (type default))
   )
@@
     (stroke (width 0) (type default))
   )
-  (wire (pts (xy 54.61 35.56) (xy 54.61 38.1))
-    (stroke (width 0) (type default))
-  )
   (wire (pts (xy 107.95 68.58) (xy 107.95 72.39))
     (stroke (width 0) (type default))
   )
-  (wire (pts (xy 54.61 48.26) (xy 58.42 48.26))
-    (stroke (width 0) (type default))
-  )
   (wire (pts (xy 110.49 91.44) (xy 96.52 91.44))
     (stroke (width 0) (type default))
   )
-  (wire (pts (xy 54.61 45.72) (xy 54.61 48.26))
-    (stroke (width 0) (type default))
-  )
   (wire (pts (xy 120.65 63.5) (xy 96.52 63.5))
     (stroke (width 0) (type default))
@@
   )
   (wire (pts (xy 101.6 44.45) (xy 115.57 44.45))
+    (stroke (width 0) (type default))
+  )
+  (wire (pts (xy 127 44.45) (xy 137.16 44.45))
     (stroke (width 0) (type default))
   )
@@
     )
   )
-  (global_label "Vmot" (shape input) (at 130.81 44.45 0) (fields_autoplaced)
+  (global_label "Vmot" (shape input) (at 137.16 44.45 0) (fields_autoplaced)
     (effects (font (size 1.27 1.27)) (justify left))
-    (property "Intersheetrefs" "${INTERSHEET_REFS}" (at 138.3724 44.45 0)
+    (property "Intersheetrefs" "${INTERSHEET_REFS}" (at 144.7224 44.45 0)
       (effects (font (size 1.27 1.27)) (justify left) hide)
     )
@@
     )
   )
-  (symbol (lib_id "power:GND") (at 48.26 48.26 270) (unit 1)
-    (in_bom yes) (on_board yes) (dnp no) (fields_autoplaced)
-    (property "Reference" "#PWR063" (at 41.91 48.26 0)
-      (effects (font (size 1.27 1.27)) hide)
-    )
-    (property "Value" "GND" (at 44.45 48.895 90)
-      (effects (font (size 1.27 1.27)) (justify right))
-    )
-    (property "Footprint" "" (at 48.26 48.26 0)
-      (effects (font (size 1.27 1.27)) hide)
-    )
-    (property "Datasheet" "" (at 48.26 48.26 0)
-      (effects (font (size 1.27 1.27)) hide)
-    )
-    (pin "1")
-    (instances
-      (project "PCB_evenwicht"
-        (path "/1568d5f0-bcdb-494d-bbf5-b93d65138b4f/0fee5d6f-552e-4af4-870f-decaeb093c62"
-          (reference "#PWR063") (unit 1)
-        )
-      )
-    )
-  )
   (symbol (lib_id "Device:R_Potentiometer") (at 40.64 86.36 0) (unit 1)
     (in_bom yes) (on_board yes) (dnp no) (fields_autoplaced)
@@
     )
   )
-  (symbol (lib_id "power:+3.3V") (at 54.61 35.56 0) (unit 1)
-    (in_bom yes) (on_board yes) (dnp no) (fields_autoplaced)
-    (property "Reference" "#PWR028" (at 54.61 39.37 0)
-      (effects (font (size 1.27 1.27)) hide)
-    )
-    (property "Value" "+3.3V" (at 54.61 31.75 0)
-      (effects (font (size 1.27 1.27)))
-    )
-    (property "Footprint" "" (at 54.61 35.56 0)
-      (effects (font (size 1.27 1.27)) hide)
-    )
-    (property "Datasheet" "" (at 54.61 35.56 0)
-      (effects (font (size 1.27 1.27)) hide)
-    )
-    (pin "1")
-    (instances
-      (project "PCB_evenwicht"
-        (path "/1568d5f0-bcdb-494d-bbf5-b93d65138b4f"
-          (reference "#PWR028") (unit 1)
-        )
-        (path "/1568d5f0-bcdb-494d-bbf5-b93d65138b4f/de18e6c3-6c35-4eb3-86ab-f4d9b06c1c30"
-          (reference "#PWR028") (unit 1)
-        )
-        (path "/1568d5f0-bcdb-494d-bbf5-b93d65138b4f/0fee5d6f-552e-4af4-870f-decaeb093c62"
-          (reference "#PWR039") (unit 1)
-        )
-      )
-    )
-  )
   (symbol (lib_id "power:GND") (at 101.6 36.83 180) (unit 1)
     (in_bom yes) (on_board yes) (dnp no) (fields_autoplaced)
@@
     )
   )
+  (symbol (lib_id "power:+3.3V") (at 48.26 48.26 0) (unit 1)
+    (in_bom yes) (on_board yes) (dnp no) (fields_autoplaced)
+    (property "Reference" "#PWR028" (at 48.26 52.07 0)
+      (effects (font (size 1.27 1.27)) hide)
+    )
+    (property "Value" "+3.3V" (at 48.26 44.45 0)
+      (effects (font (size 1.27 1.27)))
+    )
+    (property "Footprint" "" (at 48.26 48.26 0)
+      (effects (font (size 1.27 1.27)) hide)
+    )
+    (property "Datasheet" "" (at 48.26 48.26 0)
+      (effects (font (size 1.27 1.27)) hide)
+    )
+    (pin "1")
+    (instances
+      (project "PCB_evenwicht"
+        (path "/1568d5f0-bcdb-494d-bbf5-b93d65138b4f/0fee5d6f-552e-4af4-870f-decaeb093c62"
+          (reference "#PWR028") (unit 1)
+        )
+      )
+    )
+  )
   (symbol (lib_id "power:+3.3V") (at 40.64 82.55 0) (unit 1)
     (in_bom yes) (on_board yes) (dnp no) (fields_autoplaced)
@@
         (path "/1568d5f0-bcdb-494d-bbf5-b93d65138b4f/0fee5d6f-552e-4af4-870f-decaeb093c62"
           (reference "#PWR060") (unit 1)
-        )
-      )
-    )
-  )
-  (symbol (lib_id "Device:R") (at 54.61 41.91 180) (unit 1)
-    (in_bom yes) (on_board yes) (dnp no)
-    (property "Reference" "R8" (at 57.15 41.275 0)
-      (effects (font (size 1.27 1.27)) (justify right))
-    )
-    (property "Value" "100K" (at 57.15 43.18 0)
-      (effects (font (size 1.27 1.27)) (justify right))
-    )
-    (property "Footprint" "Resistor_SMD:R_0805_2012Metric_Pad1.20x1.40mm_HandSolder" (at 56.388 41.91 90)
-      (effects (font (size 1.27 1.27)) hide)
-    )
-    (property "Datasheet" "~" (at 54.61 41.91 0)
-      (effects (font (size 1.27 1.27)) hide)
-    )
-    (pin "1")
-    (pin "2")
-    (instances
-      (project "PCB_evenwicht"
-        (path "/1568d5f0-bcdb-494d-bbf5-b93d65138b4f"
-          (reference "R8") (unit 1)
-        )
-        (path "/1568d5f0-bcdb-494d-bbf5-b93d65138b4f/de18e6c3-6c35-4eb3-86ab-f4d9b06c1c30"
-          (reference "R8") (unit 1)
-        )
-        (path "/1568d5f0-bcdb-494d-bbf5-b93d65138b4f/0fee5d6f-552e-4af4-870f-decaeb093c62"
-          (reference "R12") (unit 1)
-        )
-      )
-      (project "a4988"
-        (path "/33277f75-9959-42fa-8608-f9642a2ecd81"
-          (reference "R?") (unit 1)
         )
       )
@@
         (path "/1568d5f0-bcdb-494d-bbf5-b93d65138b4f/0fee5d6f-552e-4af4-870f-decaeb093c62"
           (reference "#PWR056") (unit 1)
+        )
+      )
+    )
+  )
+  (symbol (lib_id "Device:C_Polarized") (at 127 40.64 180) (unit 1)
+    (in_bom yes) (on_board yes) (dnp no) (fields_autoplaced)
+    (property "Reference" "C19" (at 130.81 40.894 0)
+      (effects (font (size 1.27 1.27)) (justify right))
+    )
+    (property "Value" "47uF" (at 130.81 43.434 0)
+      (effects (font (size 1.27 1.27)) (justify right))
+    )
+    (property "Footprint" "Capacitor_SMD:CP_Elec_6.3x5.9" (at 126.0348 36.83 0)
+      (effects (font (size 1.27 1.27)) hide)
+    )
+    (property "Datasheet" "~" (at 127 40.64 0)
+      (effects (font (size 1.27 1.27)) hide)
+    )
+    (pin "1")
+    (pin "2")
+    (instances
+      (project "PCB_evenwicht"
+        (path "/1568d5f0-bcdb-494d-bbf5-b93d65138b4f/0fee5d6f-552e-4af4-870f-decaeb093c62"
+          (reference "C19") (unit 1)
         )
       )
@@
         (path "/1568d5f0-bcdb-494d-bbf5-b93d65138b4f/0fee5d6f-552e-4af4-870f-decaeb093c62"
           (reference "#PWR040") (unit 1)
+        )
+      )
+    )
+  )
+  (symbol (lib_id "power:GND") (at 58.42 96.52 270) (unit 1)
+    (in_bom yes) (on_board yes) (dnp no) (fields_autoplaced)
+    (property "Reference" "#PWR039" (at 52.07 96.52 0)
+      (effects (font (size 1.27 1.27)) hide)
+    )
+    (property "Value" "GND" (at 54.61 97.155 90)
+      (effects (font (size 1.27 1.27)) (justify right))
+    )
+    (property "Footprint" "" (at 58.42 96.52 0)
+      (effects (font (size 1.27 1.27)) hide)
+    )
+    (property "Datasheet" "" (at 58.42 96.52 0)
+      (effects (font (size 1.27 1.27)) hide)
+    )
+    (pin "1")
+    (instances
+      (project "PCB_evenwicht"
+        (path "/1568d5f0-bcdb-494d-bbf5-b93d65138b4f/0fee5d6f-552e-4af4-870f-decaeb093c62"
+          (reference "#PWR039") (unit 1)
         )
       )
@@
         )
       )
+    )
+  )
+  (symbol (lib_id "power:GND") (at 127 36.83 180) (unit 1)
+    (in_bom yes) (on_board yes) (dnp no) (fields_autoplaced)
+    (property "Reference" "#PWR065" (at 127 30.48 0)
+      (effects (font (size 1.27 1.27)) hide)
+    )
+    (property "Value" "GND" (at 127 33.02 0)
+      (effects (font (size 1.27 1.27)))
+    )
+    (property "Footprint" "" (at 127 36.83 0)
+      (effects (font (size 1.27 1.27)) hide)
+    )
+    (property "Datasheet" "" (at 127 36.83 0)
+      (effects (font (size 1.27 1.27)) hide)
+    )
+    (pin "1")
+    (instances
+      (project "PCB_evenwicht"
+        (path "/1568d5f0-bcdb-494d-bbf5-b93d65138b4f/0fee5d6f-552e-4af4-870f-decaeb093c62"
+          (reference "#PWR065") (unit 1)
+        )
+      )

Commit message: goed
Parts:
- C17: footprint Capacitor_SMD:C_1206_3216Metric_Pad1.33x1.80mm_HandSolder -> Capacitor_SMD:C_0805_2012Metric_Pad1.18x1.45mm_HandSolder
Connections:
- net +3.3V: now also IC1.12 (~{RESET})
- net GND: no longer IC1.12 (~{RESET})
Changed lines of the file:
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@@
+    (stroke (width 0) (type default))
+  )
+  (wire (pts (xy 49.53 66.04) (xy 58.42 66.04))
     (stroke (width 0) (type default))
   )
@@
     )
   )
+  (symbol (lib_id "power:+3.3V") (at 49.53 66.04 0) (unit 1)
+    (in_bom yes) (on_board yes) (dnp no) (fields_autoplaced)
+    (property "Reference" "#PWR063" (at 49.53 69.85 0)
+      (effects (font (size 1.27 1.27)) hide)
+    )
+    (property "Value" "+3.3V" (at 49.53 62.23 0)
+      (effects (font (size 1.27 1.27)))
+    )
+    (property "Footprint" "" (at 49.53 66.04 0)
+      (effects (font (size 1.27 1.27)) hide)
+    )
+    (property "Datasheet" "" (at 49.53 66.04 0)
+      (effects (font (size 1.27 1.27)) hide)
+    )
+    (pin "1")
+    (instances
+      (project "PCB_evenwicht"
+        (path "/1568d5f0-bcdb-494d-bbf5-b93d65138b4f/0fee5d6f-552e-4af4-870f-decaeb093c62"
+          (reference "#PWR063") (unit 1)
+        )
+      )
+    )
+  )
   (symbol (lib_id "power:GND") (at 129.54 66.04 0) (unit 1)
     (in_bom yes) (on_board yes) (dnp no) (fields_autoplaced)
@@
         (path "/33277f75-9959-42fa-8608-f9642a2ecd81"
           (reference "#PWR?") (unit 1)
-        )
-      )
-    )
-  )
-  (symbol (lib_id "power:GND") (at 58.42 66.04 270) (unit 1)
-    (in_bom yes) (on_board yes) (dnp no) (fields_autoplaced)
-    (property "Reference" "#PWR064" (at 52.07 66.04 0)
-      (effects (font (size 1.27 1.27)) hide)
-    )
-    (property "Value" "GND" (at 54.61 66.675 90)
-      (effects (font (size 1.27 1.27)) (justify right))
-    )
-    (property "Footprint" "" (at 58.42 66.04 0)
-      (effects (font (size 1.27 1.27)) hide)
-    )
-    (property "Datasheet" "" (at 58.42 66.04 0)
-      (effects (font (size 1.27 1.27)) hide)
-    )
-    (pin "1")
-    (instances
-      (project "PCB_evenwicht"
-        (path "/1568d5f0-bcdb-494d-bbf5-b93d65138b4f/0fee5d6f-552e-4af4-870f-decaeb093c62"
-          (reference "#PWR064") (unit 1)
         )
       )
@@
       (effects (font (size 1.27 1.27)) (justify left))
     )
-    (property "Footprint" "Capacitor_SMD:C_1206_3216Metric_Pad1.33x1.80mm_HandSolder" (at 116.5352 44.45 0)
-      (effects (font (size 1.27 1.27)) hide)
-    )
+    (property "Footprint" "Capacitor_SMD:C_0805_2012Metric_Pad1.18x1.45mm_HandSolder" (at 116.5352 44.45 0)
+      (effects (font (size 1.27 1.27)) hide)
+    )
