File: PCB_evenwichtsdoolhof/PCB_evenwicht.kicad_pcb (KiCad board)
At the start: 2 copper layers, 66.5 x 56.6 mm, 59 parts, among them IC1 A4988SETTR-T, IC2 A4988SETTR-T, J1 Barrel_Jack, J2 Conn_01x04_Pin, J3 Switchy, J4 Conn_01x04_Pin, J5 POTy, J6 Conn_01x04_Pin, J7 Switchx, J8 POTx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

Commit message: File Restructuring
Restructuring and removing old files
+ cleaning up code
Connections:
- J5 pad 2: A9 -> GPIO35
- J8 pad 2: A8 -> GPIO34
- U1 pad 6: unconnected-(U1-IO34-Pad6) -> GPIO34
- U1 pad 7: unconnected-(U1-IO35-Pad7) -> GPIO35
Routing:
- net GPIO35: track 0.00 -> 27.1 mm, vias 0 -> 1
- net GPIO34: track 0.00 -> 23.3 mm, vias 0 -> 1
- net A9: track 23.1 -> 0.00 mm, vias 1 -> 0
- net A8: track 18.5 -> 0.00 mm, vias 1 -> 0
- net GND: vias 34 -> 35
Other:
- board text added: "Emiel Dever & Jonathan Gheysens IB3 V1.2"
- board text removed: "Emiel Dever & Jonathan Gheysens IB3 V1.1"
Changed lines of the file:
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@@
   (net 71 "unconnected-(U1-SENSOR_VP-Pad4)")
   (net 72 "unconnected-(U1-SENSOR_VN-Pad5)")
-  (net 73 "unconnected-(U1-IO34-Pad6)")
-  (net 74 "unconnected-(U1-IO35-Pad7)")
+  (net 73 "GPIO35")
+  (net 74 "GPIO34")
   (net 75 "MS1_2")
   (net 76 "MS2_2")
@@
       (net 72 "unconnected-(U1-SENSOR_VN-Pad5)") (pinfunction "SENSOR_VN") (pintype "input+no_connect"))
     (pad "6" smd rect (at -8.75 -1.9) (size 1.5 0.9) (layers "F.Cu" "F.Paste" "F.Mask")
-      (net 73 "unconnected-(U1-IO34-Pad6)") (pinfunction "IO34") (pintype "input+no_connect"))
+      (net 74 "GPIO34") (pinfunction "IO34") (pintype "input"))
     (pad "7" smd rect (at -8.75 -0.63) (size 1.5 0.9) (layers "F.Cu" "F.Paste" "F.Mask")
-      (net 74 "unconnected-(U1-IO35-Pad7)") (pinfunction "IO35") (pintype "input+no_connect"))
+      (net 73 "GPIO35") (pinfunction "IO35") (pintype "input"))
     (pad "8" smd rect (at -8.75 0.64) (size 1.5 0.9) (layers "F.Cu" "F.Paste" "F.Mask")
       (net 16 "A4") (pinfunction "IO32") (pintype "bidirectional"))
@@
       (net 2 "GND") (pinfunction "Pin_1") (pintype "passive"))
     (pad "2" thru_hole oval (at 0 2.54 90) (size 1.7 1.7) (drill 1) (layers "*.Cu" "*.Mask")
-      (net 18 "A8") (pinfunction "Pin_2") (pintype "passive"))
+      (net 74 "GPIO34") (pinfunction "Pin_2") (pintype "passive"))
     (pad "3" thru_hole oval (at 0 5.08 90) (size 1.7 1.7) (drill 1) (layers "*.Cu" "*.Mask")
       (net 1 "+3.3V") (pinfunction "Pin_3") (pintype "passive"))
@@
       (net 2 "GND") (pinfunction "Pin_1") (pintype "passive"))
     (pad "2" thru_hole oval (at 0 2.54 90) (size 1.7 1.7) (drill 1) (layers "*.Cu" "*.Mask")
-      (net 19 "A9") (pinfunction "Pin_2") (pintype "passive"))
+      (net 73 "GPIO35") (pinfunction "Pin_2") (pintype "passive"))
     (pad "3" thru_hole oval (at 0 5.08 90) (size 1.7 1.7) (drill 1) (layers "*.Cu" "*.Mask")
       (net 1 "+3.3V") (pinfunction "Pin_3") (pintype "passive"))
@@
     (effects (font (size 1 1) (thickness 0.1)) (justify left bottom))
   )
-  (gr_text "Emiel Dever &\nJonathan Gheysens\nIB3 V1.1" (at 154.1272 100.9396) (layer "F.SilkS")
+  (gr_text "Emiel Dever &\nJonathan Gheysens\nIB3 V1.2" (at 154.1272 100.9396) (layer "F.SilkS")
     (effects (font (size 1 1) (thickness 0.1)) (justify left bottom))
   )
@@
   (via (at 161.1376 81.28) (size 0.6) (drill 0.3) (layers "F.Cu" "B.Cu") (net 2))
   (via (at 159.9184 81.8896) (size 0.6) (drill 0.3) (layers "F.Cu" "B.Cu") (net 2))
-  (via (at 113.7412 63.2968) (size 0.6) (drill 0.3) (layers "F.Cu" "B.Cu") (free) (net 2))
+  (via (at 112.2172 67.9704) (size 0.6) (drill 0.3) (layers "F.Cu" "B.Cu") (free) (net 2))
   (via (at 160.7312 58.928) (size 0.6) (drill 0.3) (layers "F.Cu" "B.Cu") (net 2))
   (via (at 161.9504 58.3184) (size 0.6) (drill 0.3) (layers "F.Cu" "B.Cu") (net 2))
@@
   (via (at 151.892 71.7804) (size 0.6) (drill 0.3) (layers "F.Cu" "B.Cu") (free) (net 2))
   (via (at 165.5244 63.754002) (size 0.6) (drill 0.3) (layers "F.Cu" "B.Cu") (free) (net 2))
+  (via (at 118.9736 69.596) (size 0.6) (drill 0.3) (layers "F.Cu" "B.Cu") (free) (net 2))
   (via (at 167.2336 51.5112) (size 0.6) (drill 0.3) (layers "F.Cu" "B.Cu") (free) (net 2))
   (via (at 161.9504 58.928) (size 0.6) (drill 0.3) (layers "F.Cu" "B.Cu") (net 2))
@@
   (segment (start 147.5232 75.7428) (end 128.016 75.7428) (width 0.3) (layer "B.Cu") (net 17))
   (segment (start 128.016 75.7428) (end 116.332 64.0588) (width 0.3) (layer "B.Cu") (net 17))
-  (segment (start 116.345 65.365) (end 114.808 65.365) (width 0.3) (layer "F.Cu") (net 18))
-  (via (at 114.807998 65.365002) (size 0.6) (drill 0.3) (layers "F.Cu" "B.Cu") (net 18))
-  (segment (start 110.236 80.264) (end 110.236 69.596) (width 0.3) (layer "B.Cu") (net 18))
-  (segment (start 114.720998 65.365002) (end 114.807998 65.365002) (width 0.2) (layer "B.Cu") (net 18))
-  (segment (start 110.236 69.596) (end 114.466998 65.365002) (width 0.3) (layer "B.Cu") (net 18))
-  (segment (start 114.466998 65.365002) (end 114.720998 65.365002) (width 0.3) (layer "B.Cu") (net 18))
-  (segment (start 114.808002 66.635) (end 116.345 66.635) (width 0.3) (layer "F.Cu") (net 19))
-  (segment (start 114.173 66.802) (end 114.808002 66.635) (width 0.3) (layer "F.Cu") (net 19))
-  (segment (start 114.173 66.802) (end 114.808 66.635002) (width 0.3) (layer "F.Cu") (net 19))
-  (via (at 114.173 66.802) (size 0.6) (drill 0.3) (layers "F.Cu" "B.Cu") (net 19))
-  (segment (start 114.1476 66.8274) (end 114.173 66.802) (width 0.3) (layer "B.Cu") (net 19))
-  (segment (start 114.1476 81.9404) (end 114.1476 66.8274) (width 0.3) (layer "B.Cu") (net 19))
-  (segment (start 112.522 82.55) (end 113.538 82.55) (width 0.3) (layer "B.Cu") (net 19))
-  (segment (start 113.538 82.55) (end 114.1476 81.9404) (width 0.3) (layer "B.Cu") (net 19))
-  (segment (start 110.236 84.836) (end 112.522 82.55) (width 0.3) (layer "B.Cu") (net 19))
   (segment (start 116.345 67.905) (end 114.823866 67.905) (width 0.3) (layer "F.Cu") (net 20))
   (segment (start 114.823866 67.905) (end 114.807998 67.920868) (width 0.3) (layer "F.Cu") (net 20))
@@
   (segment (start 113.014 58.182) (end 109.474 61.722) (width 0.4) (layer "F.Cu") (net 70))
   (segment (start 113.03 58.182) (end 113.014 58.182) (width 0.4) (layer "F.Cu") (net 70))
+  (segment (start 115.1782 61.555) (end 116.345 61.555) (width 0.3) (layer "F.Cu") (net 73))
+  (segment (start 114.8588 61.8744) (end 115.1782 61.555) (width 0.3) (layer "F.Cu") (net 73))
+  (via (at 114.8588 61.8744) (size 0.6) (drill 0.3) (layers "F.Cu" "B.Cu") (net 73))
+  (segment (start 110.236 84.836) (end 112.522 82.55) (width 0.3) (layer "B.Cu") (net 73))
+  (segment (start 114.1476 62.5856) (end 114.8588 61.8744) (width 0.3) (layer "B.Cu") (net 73))
+  (segment (start 112.522 82.55) (end 113.538 82.55) (width 0.3) (layer "B.Cu") (net 73))
+  (segment (start 113.538 82.55) (end 114.1476 81.9404) (width 0.3) (layer "B.Cu") (net 73))
+  (segment (start 114.1476 81.9404) (end 114.1476 62.5856) (width 0.3) (layer "B.Cu") (net 73))
+  (segment (start 116.2796 60.3504) (end 116.345 60.285) (width 0.3) (layer "F.Cu") (net 74))
+  (segment (start 114.9096 60.3504) (end 116.2796 60.3504) (width 0.3) (layer "F.Cu") (net 74))
+  (via (at 114.9096 60.3504) (size 0.6) (drill 0.3) (layers "F.Cu" "B.Cu") (net 74))
+  (segment (start 110.236 80.264) (end 110.236 65.024) (width 0.3) (layer "B.Cu") (net 74))
+  (segment (start 110.236 65.024) (end 114.9096 60.3504) (width 0.3) (layer "B.Cu") (net 74))
   (segment (start 163.267 73.481) (end 164.261 72.487) (width 0.3) (layer "F.Cu") (net 75))
   (segment (start 163.267 74.803) (end 163.267 73.481) (width 0.3) (layer "F.Cu") (net 75))
