File: PCB_evenwichtsdoolhof/PCB_evenwicht.kicad_sch (KiCad schematic)
At the start: 17 parts, among them J1 Barrel_Jack, J3 Switchy, J5 POTy, J7 Switchx, J8 POTx, J9 Switch_einde, U2 AMS1117-3.3, U3 MP1584

Commit message: File Restructuring
Restructuring and removing old files
+ cleaning up code
Connections:
- net A8 renamed GPIO34
- net A9 renamed GPIO35
Changed lines of the file:
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@@
     )
   )
-  (global_label "A9" (shape input) (at 127 68.58 0) (fields_autoplaced)
+  (global_label "GPIO35" (shape input) (at 127 68.58 0) (fields_autoplaced)
     (effects (font (size 1.27 1.27)) (justify left))
-    (property "Intersheetrefs" "${INTERSHEET_REFS}" (at 132.2039 68.58 0)
+    (property "Intersheetrefs" "${INTERSHEET_REFS}" (at 136.8001 68.58 0)
       (effects (font (size 1.27 1.27)) (justify left) hide)
     )
   )
-  (global_label "A8" (shape input) (at 127 102.87 0) (fields_autoplaced)
+  (global_label "GPIO34" (shape input) (at 127 102.87 0) (fields_autoplaced)
     (effects (font (size 1.27 1.27)) (justify left))
-    (property "Intersheetrefs" "${INTERSHEET_REFS}" (at 132.2039 102.87 0)
+    (property "Intersheetrefs" "${INTERSHEET_REFS}" (at 136.8001 102.87 0)
       (effects (font (size 1.27 1.27)) (justify left) hide)
     )
